File: backplane.kicad_pcb (KiCad board)
At the start: 2 copper layers, 88.9 x 83.8 mm, 15 parts, among them J1 I2C, J2 GPS, J3 SERIAL_HEADER, J4 PWR_HEADER, Q1 Q_NMOS_DGS, Q2 Q_NMOS_DGS, Q3 Q_NMOS_DGS, U1 Raspberry_Pi_2_3, U2 IC880A-SPI

Commit message: More ground connections and thicker power tracks
Parts:
- J1: value I2C -> I2C_HEADER
- J2: value GPS -> GPS_HEADER
Connections:
- J1 pad 4: Net-(J1-Pad4) -> /3.3V
- J1 pad 5: Net-(J1-Pad5) -> /5V
- J2 pad 4: Net-(J2-Pad4) -> /3.3V
- J2 pad 5: Net-(J1-Pad5) -> /5V
- J4 pad 2: Net-(J4-Pad2) -> /5V
- R1 pad 2: Net-(J1-Pad4) -> /3.3V
- R2 pad 2: Net-(J1-Pad4) -> /3.3V
- R3 pad 2: Net-(J1-Pad4) -> /3.3V
- U1 pad 1: Net-(J1-Pad4) -> /3.3V
- U1 pad 17: Net-(J2-Pad4) -> /3.3V
- U1 pad 2: Net-(J4-Pad2) -> /5V
- U1 pad 4: Net-(J1-Pad5) -> /5V
- U2 pad 1: Net-(U2-Pad1) -> GND
- U2 pad 12: Net-(U2-Pad12) -> GND
- U2 pad 20: Net-(U2-Pad20) -> GND
- U2 pad 21: Net-(J4-Pad2) -> /5V
Routing:
- net /3.3V: track 0.00 -> 274.1 mm, vias 0 -> 5
- net /5V: track 0.00 -> 237.4 mm, vias 0 -> 3
- net Net-(J1-Pad4): track 172.6 -> 0.00 mm, vias 2 -> 0
- net Net-(J1-Pad5): track 133.7 -> 0.00 mm, vias 1 -> 0
- net Net-(J4-Pad2): track 103.8 -> 0.00 mm, vias 2 -> 0
- net Net-(J2-Pad4): track 101.5 -> 0.00 mm, vias 3 -> 0
Other:
- net class Power added: clearance 0.2, trace_width 0.8, via_dia 1, via_drill 0.8

Commit message: Fixes
Connections:
- U1 pad 6: GND -> Net-(U1-Pad6)
Routing:
- net GND: track 0.00 -> 13.4 mm
- net (no net): track 0.00 -> 4.57 mm
- net /5V: track 237.4 -> 240.0 mm
- net /3.3V: vias 5 -> 6
Changed lines of the file:
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@@
 (kicad_pcb (version 4) (host pcbnew 4.0.5)
   (general
-    (links 51)
-    (no_connects 4)
-    (area 100.889999 69.139999 189.940001 153.110001)
+    (links 50)
+    (no_connects 0)
+    (area 86.995 57.785 200.025001 156.845001)
     (thickness 1.6)
     (drawings 7)
-    (tracks 181)
+    (tracks 196)
     (zones 0)
     (modules 15)
-    (nets 52)
+    (nets 53)
   )
   (page A4)
@@
   (net 50 /3.3V)
   (net 51 /5V)
+  (net 52 "Net-(U1-Pad6)")
   (net_class Default "This is the default net class."
     (clearance 0.2)
@@
     (add_net "Net-(U1-Pad35)")
     (add_net "Net-(U1-Pad37)")
+    (add_net "Net-(U1-Pad6)")
     (add_net "Net-(U1-Pad7)")
     (add_net "Net-(U2-Pad10)")
@@
       (net 8 "Net-(J1-Pad2)"))
     (pad 6 thru_hole oval (at 2.54 5.08 270) (size 1.7 1.7) (drill 1) (layers *.Cu *.Mask)
-      (net 16 GND))
+      (net 52 "Net-(U1-Pad6)"))
     (pad 7 thru_hole oval (at 0 7.62 270) (size 1.7 1.7) (drill 1) (layers *.Cu *.Mask)
       (net 19 "Net-(U1-Pad7)"))
@@
   (gr_line (start 179.07 153.035) (end 100.965 153.035) (angle 90) (layer Edge.Cuts) (width 0.15))
   (gr_line (start 179.07 153.035) (end 187.96 153.035) (angle 90) (layer Edge.Cuts) (width 0.15))
+  (segment (start 182.499 139.065) (end 182.499 137.541) (width 0.8) (layer B.Cu) (net 0))
+  (segment (start 182.499 140.589) (end 182.499 139.065) (width 0.8) (layer F.Cu) (net 0))
+  (segment (start 182.499 142.113) (end 182.499 140.589) (width 0.8) (layer B.Cu) (net 0))
   (segment (start 122.555 128.365) (end 106.84 128.365) (width 0.25) (layer F.Cu) (net 1))
   (segment (start 106.84 128.365) (end 106.68 128.525) (width 0.25) (layer F.Cu) (net 1))
@@
   (segment (start 102.87 118.11) (end 102.235 118.745) (width 0.25) (layer F.Cu) (net 15))
   (segment (start 107.635 113.345) (end 102.87 118.11) (width 0.25) (layer F.Cu) (net 15))
+  (segment (start 157.226 147.066) (end 157.353 147.066) (width 0.25) (layer F.Cu) (net 16))
+  (segment (start 157.353 147.066) (end 158.623 145.796) (width 0.25) (layer F.Cu) (net 16))
+  (segment (start 158.623 145.796) (end 161.036 145.796) (width 0.25) (layer F.Cu) (net 16))
+  (segment (start 161.036 145.796) (end 162.306 144.526) (width 0.25) (layer F.Cu) (net 16))
+  (segment (start 180.34 147.32) (end 182.372 147.32) (width 0.8) (layer F.Cu) (net 16))
+  (segment (start 182.499 147.193) (end 182.499 142.113) (width 0.8) (layer F.Cu) (net 16))
+  (segment (start 182.372 147.32) (end 182.499 147.193) (width 0.8) (layer F.Cu) (net 16))
   (segment (start 112.165 123.505) (end 107.635 123.505) (width 0.25) (layer F.Cu) (net 17))
   (segment (start 124.587 149.225) (end 126.746 147.066) (width 0.25) (layer F.Cu) (net 17))
@@
   (segment (start 134.3611 135.6536) (end 134.3611 144.5211) (width 0.25) (layer F.Cu) (net 35) (status 10))
   (segment (start 134.3611 144.5211) (end 134.366 144.526) (width 0.25) (layer F.Cu) (net 35))
+  (via (at 118.999 106.585) (size 1) (drill 0.8) (layers F.Cu B.Cu) (net 50))
+  (segment (start 118.999 106.585) (end 118.999 106.553) (width 0.8) (layer B.Cu) (net 50))
   (segment (start 109.347 100.965) (end 104.775 100.965) (width 0.8) (layer F.Cu) (net 50))
-  (segment (start 122.555 106.585) (end 114.967 106.585) (width 0.8) (layer F.Cu) (net 50))
+  (segment (start 122.555 106.585) (end 118.999 106.585) (width 0.8) (layer F.Cu) (net 50))
+  (segment (start 118.999 106.585) (end 114.967 106.585) (width 0.8) (layer F.Cu) (net 50))
   (segment (start 114.967 106.585) (end 109.347 100.965) (width 0.8) (layer F.Cu) (net 50))
   (segment (start 175.387 131.953) (end 177.927 134.493) (width 0.8) (layer F.Cu) (net 50))
@@
   (segment (start 126.619 106.553) (end 126.587 106.585) (width 0.8) (layer F.Cu) (net 50))
   (segment (start 156.591 113.157) (end 155.829 112.395) (width 0.8) (layer F.Cu) (net 50))
-  (segment (start 118.999 91.821) (end 118.999 90.297) (width 0.25) (layer F.Cu) (net 50))
-  (segment (start 152.146 140.208) (end 149.479 137.541) (width 0.25) (layer B.Cu) (net 50))
-  (segment (start 149.479 137.541) (end 132.969 137.541) (width 0.25) (layer B.Cu) (net 50))
-  (via (at 132.969 137.541) (size 0.6) (drill 0.4) (layers F.Cu B.Cu) (net 50))
-  (segment (start 132.969 137.541) (end 129.159 137.541) (width 0.25) (layer F.Cu) (net 50))
-  (via (at 129.159 137.541) (size 0.6) (drill 0.4) (layers F.Cu B.Cu) (net 50))
-  (segment (start 129.159 137.541) (end 123.317 137.541) (width 0.25) (layer B.Cu) (net 50))
-  (segment (start 123.317 137.541) (end 122.301 136.525) (width 0.25) (layer B.Cu) (net 50))
-  (segment (start 122.301 136.525) (end 122.301 134.747) (width 0.25) (layer B.Cu) (net 50))
-  (segment (start 122.301 134.747) (end 118.999 131.445) (width 0.25) (layer B.Cu) (net 50))
-  (segment (start 118.999 131.445) (end 118.999 97.409) (width 0.25) (layer B.Cu) (net 50))
-  (via (at 118.999 97.409) (size 0.6) (drill 0.4) (layers F.Cu B.Cu) (net 50))
-  (segment (start 118.999 97.409) (end 118.999 91.821) (width 0.25) (layer F.Cu) (net 50))
-  (segment (start 152.146 144.526) (end 152.146 140.208) (width 0.25) (layer B.Cu) (net 50))
-  (segment (start 109.347 80.645) (end 104.775 80.645) (width 0.25) (layer F.Cu) (net 50))
-  (segment (start 118.999 90.297) (end 109.347 80.645) (width 0.25) (layer F.Cu) (net 50))
+  (segment (start 118.999 91.821) (end 118.999 90.297) (width 0.8) (layer F.Cu) (net 50))
+  (segment (start 118.999 90.297) (end 109.347 80.645) (width 0.8) (layer F.Cu) (net 50))
+  (segment (start 109.347 80.645) (end 104.775 80.645) (width 0.8) (layer F.Cu) (net 50))
+  (segment (start 152.146 144.526) (end 152.146 140.208) (width 0.8) (layer B.Cu) (net 50))
+  (segment (start 118.999 131.445) (end 118.999 106.553) (width 0.8) (layer B.Cu) (net 50))
+  (segment (start 122.301 134.747) (end 118.999 131.445) (width 0.8) (layer B.Cu) (net 50))
+  (segment (start 122.301 136.525) (end 122.301 134.747) (width 0.8) (layer B.Cu) (net 50))
+  (segment (start 123.317 137.541) (end 122.301 136.525) (width 0.8) (layer B.Cu) (net 50))
+  (segment (start 129.159 137.541) (end 123.317 137.541) (width 0.8) (layer B.Cu) (net 50))
+  (via (at 129.159 137.541) (size 1) (drill 0.8) (layers F.Cu B.Cu) (net 50))
+  (segment (start 132.969 137.541) (end 129.159 137.541) (width 0.8) (layer F.Cu) (net 50))
+  (via (at 132.969 137.541) (size 1) (drill 0.8) (layers F.Cu B.Cu) (net 50))
+  (segment (start 149.479 137.541) (end 132.969 137.541) (width 0.8) (layer B.Cu) (net 50))
+  (segment (start 152.146 140.208) (end 149.479 137.541) (width 0.8) (layer B.Cu) (net 50))
+  (segment (start 118.999 97.409) (end 118.999 91.821) (width 0.8) (layer F.Cu) (net 50))
+  (via (at 118.999 97.409) (size 1) (drill 0.8) (layers F.Cu B.Cu) (net 50))
+  (segment (start 118.999 106.553) (end 118.999 97.409) (width 0.8) (layer B.Cu) (net 50) (status 2))
+  (segment (start 169.926 147.066) (end 172.466 147.066) (width 0.8) (layer F.Cu) (net 51))
   (segment (start 104.775 103.505) (end 102.87 103.505) (width 0.8) (layer B.Cu) (net 51))
   (segment (start 104.775 83.312) (end 104.775 83.185) (width 0.25) (layer B.Cu) (net 51))

Commit message: Add text to PCB
Parts:
- added G***: LOGO, oshw-logos:OSHW_MASK_7MM, F.Cu at (173.4, 83.2)
Other:
- board text added: "iC880A Backplane v1.0 coredump.ch / adnexo.ch 2017"
- board text added: "open source hardware"
Changed lines of the file:
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@@
     (area 86.995 57.785 200.025001 156.845001)
     (thickness 1.6)
-    (drawings 7)
+    (drawings 9)
     (tracks 196)
     (zones 0)
-    (modules 15)
+    (modules 16)
     (nets 53)
   )
@@
     )
   )
+  (module oshw-logos:OSHW_MASK_7MM (layer F.Cu)
+    (at 173.355 83.185 270)
+    (fp_text reference G*** (at 0 3.71094 270) (layer F.Mask) hide
+      (effects (font (size 0.3175 0.3175) (thickness 0.0635)))
+    )
+    (fp_text value LOGO (at 0 -3.71094 270) (layer F.Mask) hide
+      (effects (font (size 0.3175 0.3175) (thickness 0.0635)))
+    )
+    (fp_poly (pts (xy -2.1209 3.14452) (xy -2.08534 3.1242) (xy -2.00152 3.0734) (xy -1.88468 2.9972)
+      (xy -1.74752 2.90322) (xy -1.60782 2.80924) (xy -1.49606 2.73304) (xy -1.41478 2.68224)
+      (xy -1.38176 2.66446) (xy -1.36398 2.66954) (xy -1.29794 2.70256) (xy -1.20142 2.75082)
+      (xy -1.14808 2.7813) (xy -1.05918 2.8194) (xy -1.016 2.82702) (xy -1.00838 2.81432)
+      (xy -0.97536 2.74574) (xy -0.92456 2.63144) (xy -0.85852 2.48158) (xy -0.78486 2.30378)
+      (xy -0.70358 2.11074) (xy -0.6223 1.91516) (xy -0.54356 1.72974) (xy -0.47498 1.5621)
+      (xy -0.42164 1.42494) (xy -0.38354 1.33096) (xy -0.37084 1.29032) (xy -0.37592 1.2827)
+      (xy -0.4191 1.23952) (xy -0.4953 1.1811) (xy -0.6604 1.04648) (xy -0.8255 0.84328)
+      (xy -0.92456 0.61214) (xy -0.95758 0.35306) (xy -0.92964 0.1143) (xy -0.83566 -0.1143)
+      (xy -0.67564 -0.32004) (xy -0.4826 -0.47244) (xy -0.254 -0.5715) (xy 0 -0.60198)
+      (xy 0.24384 -0.57404) (xy 0.47752 -0.4826) (xy 0.68326 -0.32512) (xy 0.77216 -0.22352)
+      (xy 0.89154 -0.01524) (xy 0.96012 0.20828) (xy 0.96774 0.26416) (xy 0.95758 0.51054)
+      (xy 0.88392 0.74676) (xy 0.75438 0.95758) (xy 0.57404 1.1303) (xy 0.55118 1.14554)
+      (xy 0.46736 1.20904) (xy 0.41148 1.25222) (xy 0.3683 1.28778) (xy 0.68072 2.03962)
+      (xy 0.73152 2.16154) (xy 0.81788 2.36728) (xy 0.89408 2.54508) (xy 0.9525 2.68478)
+      (xy 0.99568 2.77876) (xy 1.01346 2.81686) (xy 1.016 2.8194) (xy 1.04394 2.82448)
+      (xy 1.09982 2.80416) (xy 1.2065 2.75336) (xy 1.27508 2.7178) (xy 1.35636 2.67716)
+      (xy 1.39192 2.66446) (xy 1.4224 2.6797) (xy 1.4986 2.7305) (xy 1.61036 2.80416)
+      (xy 1.74498 2.8956) (xy 1.87452 2.9845) (xy 1.99136 3.0607) (xy 2.07772 3.11658)
+      (xy 2.11836 3.13944) (xy 2.12598 3.13944) (xy 2.16408 3.11912) (xy 2.23012 3.0607)
+      (xy 2.33426 2.96418) (xy 2.47904 2.82194) (xy 2.5019 2.79908) (xy 2.62128 2.67716)
+      (xy 2.7178 2.57556) (xy 2.7813 2.50444) (xy 2.8067 2.47142) (xy 2.8067 2.47142)
+      (xy 2.78384 2.43078) (xy 2.7305 2.34442) (xy 2.65176 2.22504) (xy 2.55524 2.08534)
+      (xy 2.30632 1.72212) (xy 2.44348 1.37922) (xy 2.48666 1.27508) (xy 2.54 1.14808)
+      (xy 2.5781 1.05664) (xy 2.59842 1.01854) (xy 2.63652 1.0033) (xy 2.7305 0.98298)
+      (xy 2.86512 0.95504) (xy 3.02768 0.92456) (xy 3.18262 0.89408) (xy 3.32232 0.86868)
+      (xy 3.42138 0.84836) (xy 3.4671 0.84074) (xy 3.47726 0.83312) (xy 3.48742 0.8128)
+      (xy 3.4925 0.76454) (xy 3.49758 0.68072) (xy 3.49758 0.5461) (xy 3.49758 0.35306)
+      (xy 3.49758 0.33274) (xy 3.49758 0.14732) (xy 3.4925 0.00254) (xy 3.48742 -0.09398)
+      (xy 3.48234 -0.13208) (xy 3.48234 -0.13208) (xy 3.43916 -0.14224) (xy 3.3401 -0.16256)
+      (xy 3.2004 -0.1905) (xy 3.0353 -0.22098) (xy 3.02514 -0.22352) (xy 2.8575 -0.25654)
+      (xy 2.72034 -0.28448) (xy 2.62382 -0.30734) (xy 2.58064 -0.32004) (xy 2.57302 -0.3302)
+      (xy 2.54 -0.39624) (xy 2.49174 -0.49784) (xy 2.4384 -0.62484) (xy 2.38252 -0.75438)
+      (xy 2.3368 -0.87122) (xy 2.30632 -0.95758) (xy 2.29616 -0.99822) (xy 2.29616 -0.99822)
+      (xy 2.32156 -1.03886) (xy 2.37744 -1.12268) (xy 2.45872 -1.24206) (xy 2.55524 -1.3843)
+      (xy 2.56286 -1.39446) (xy 2.65684 -1.53416) (xy 2.73558 -1.65354) (xy 2.78638 -1.73736)
+      (xy 2.8067 -1.77546) (xy 2.80416 -1.778) (xy 2.77368 -1.81864) (xy 2.70256 -1.89992)
+      (xy 2.60096 -2.0066) (xy 2.4765 -2.12852) (xy 2.4384 -2.16662) (xy 2.30378 -2.30124)
+      (xy 2.20726 -2.3876) (xy 2.14884 -2.43332) (xy 2.1209 -2.44348) (xy 2.1209 -2.44348)
+      (xy 2.07772 -2.41808) (xy 1.98882 -2.35966) (xy 1.86944 -2.27838) (xy 1.7272 -2.18186)
+      (xy 1.71704 -2.17678) (xy 1.57734 -2.08026) (xy 1.4605 -2.00152) (xy 1.37922 -1.94564)
+      (xy 1.34366 -1.92532) (xy 1.33604 -1.92532) (xy 1.28016 -1.94056) (xy 1.1811 -1.97612)
+      (xy 1.05664 -2.02438) (xy 0.9271 -2.07518) (xy 0.81026 -2.12598) (xy 0.72136 -2.16662)
+      (xy 0.68072 -2.18948) (xy 0.67818 -2.19202) (xy 0.66548 -2.24282) (xy 0.64008 -2.34696)
+      (xy 0.6096 -2.49174) (xy 0.57912 -2.66192) (xy 0.57404 -2.68986) (xy 0.54102 -2.85496)
+      (xy 0.51562 -2.99466) (xy 0.4953 -3.08864) (xy 0.48514 -3.12928) (xy 0.46228 -3.13436)
+      (xy 0.381 -3.13944) (xy 0.25654 -3.14198) (xy 0.10414 -3.14452) (xy -0.05334 -3.14452)
+      (xy -0.20828 -3.13944) (xy -0.34036 -3.13436) (xy -0.43434 -3.12928) (xy -0.47244 -3.12166)
+      (xy -0.47498 -3.11912) (xy -0.49022 -3.06832) (xy -0.51308 -2.96164) (xy -0.54102 -2.81686)
+      (xy -0.57404 -2.64668) (xy -0.57912 -2.6162) (xy -0.61214 -2.44856) (xy -0.64008 -2.3114)
+      (xy -0.6604 -2.21996) (xy -0.67056 -2.18186) (xy -0.6858 -2.17424) (xy -0.75438 -2.14376)
+      (xy -0.86614 -2.09804) (xy -1.0033 -2.04216) (xy -1.32334 -1.91262) (xy -1.71704 -2.18186)
+      (xy -1.7526 -2.20472) (xy -1.89484 -2.30124) (xy -2.00914 -2.37998) (xy -2.09042 -2.43078)
+      (xy -2.12344 -2.4511) (xy -2.12598 -2.44856) (xy -2.16662 -2.41554) (xy -2.24536 -2.34188)
+      (xy -2.3495 -2.23774) (xy -2.47396 -2.11582) (xy -2.5654 -2.02438) (xy -2.67462 -1.91262)
+      (xy -2.7432 -1.83896) (xy -2.77876 -1.7907) (xy -2.794 -1.76276) (xy -2.78892 -1.74498)
+      (xy -2.76352 -1.70434) (xy -2.70764 -1.61798) (xy -2.62636 -1.4986) (xy -2.52984 -1.3589)
+      (xy -2.4511 -1.24206) (xy -2.36728 -1.10998) (xy -2.3114 -1.016) (xy -2.29108 -0.97028)
+      (xy -2.29616 -0.9525) (xy -2.3241 -0.87376) (xy -2.36982 -0.75946) (xy -2.43078 -0.61976)
+      (xy -2.5654 -0.30988) (xy -2.77114 -0.26924) (xy -2.89306 -0.24638) (xy -3.06578 -0.21336)
+      (xy -3.23088 -0.18034) (xy -3.48996 -0.13208) (xy -3.50012 0.81534) (xy -3.45948 0.83312)
+      (xy -3.42138 0.84328) (xy -3.32486 0.8636) (xy -3.1877 0.89154) (xy -3.02768 0.92202)
+      (xy -2.89052 0.94742) (xy -2.75336 0.97536) (xy -2.6543 0.99314) (xy -2.60858 1.0033)
+      (xy -2.59842 1.01854) (xy -2.56286 1.08458) (xy -2.5146 1.19126) (xy -2.45872 1.31826)
+      (xy -2.40284 1.45288) (xy -2.35458 1.5748) (xy -2.32156 1.66878) (xy -2.30886 1.71704)
+      (xy -2.32664 1.7526) (xy -2.37998 1.83388) (xy -2.45618 1.95072) (xy -2.55016 2.08788)
+      (xy -2.64414 2.22504) (xy -2.72288 2.34188) (xy -2.77876 2.4257) (xy -2.80162 2.4638)
+      (xy -2.78892 2.49174) (xy -2.73558 2.55778) (xy -2.63144 2.66446) (xy -2.4765 2.81686)
+      (xy -2.4511 2.84226) (xy -2.32918 2.9591) (xy -2.22504 3.05562) (xy -2.15392 3.11912)
+      (xy -2.1209 3.14452)) (layer F.Mask) (width 0.00254))
+  )
+  (gr_text "open source hardware" (at 173.355 100.965 270) (layer F.Mask)
+    (effects (font (size 1.5 1.5) (thickness 0.3)))
+  )
+  (gr_text "iC880A Backplane v1.0\ncoredump.ch / adnexo.ch 2017" (at 183.515 93.345 270) (layer F.Mask)
+    (effects (font (size 1.5 1.5) (thickness 0.3)))
+  )
   (gr_line (start 189.865 153.035) (end 187.96 153.035) (angle 90) (layer Edge.Cuts) (width 0.15))

Commit message: Remove GPS header (fixes #1)
Parts:
- removed G***: LOGO, oshw-logos:OSHW_MASK_7MM
- removed J2: GPS_HEADER, Pin_Headers:Pin_Header_Straight_1x06_Pitch2.54mm
- J1: value I2C_HEADER -> I2C
- J3: value SERIAL_HEADER -> SER
- J4: value PWR_HEADER -> PWR
- moved D1 41.0 mm to (69.6, 112.6)
- moved D3 41.0 mm to (69.6, 92.3)
- moved Q2 41.0 mm to (76.6, 105.0)
- moved Q3 41.0 mm to (76.6, 115.2)
- moved U1 41.0 mm to (135.4, 127.0)
- moved U2 41.0 mm to (111.4, 87.5)
- moved D2 41.0 mm to (69.6, 102.5)
- moved J1 41.0 mm to (67.7, 75.8)
- moved J3 41.0 mm to (149.6, 127.3)
- moved Q1 41.0 mm to (76.6, 94.9)
- moved R1 41.0 mm to (85.5, 108.8)
- moved R2 41.0 mm to (85.5, 99.9)
- moved R3 41.0 mm to (85.5, 91.1)
- moved J4 41.0 mm to (143.3, 129.8)
Connections:
- U2 pad 24: Net-(J2-Pad3) -> GND
Routing:
- net /3.3V: track 274.1 -> 195.6 mm, vias 6 -> 0
- net Net-(J2-Pad3): track 72.7 -> 0.00 mm
- net Net-(U2-Pad26): track 66.7 -> 0.00 mm
- net Net-(U2-Pad25): track 64.5 -> 0.01 mm
- net Net-(U2-Pad23): track 31.7 -> 0.00 mm
- net /5V: track 240.0 -> 215.7 mm, vias 3 -> 1
