File: backplane.kicad_pcb (KiCad board)
At the start: 2 copper layers, 88.9 x 83.8 mm, 14 parts, among them J1 I2C, J3 SER, J4 PWR, Q1 Q_NMOS_DGS, Q2 Q_NMOS_DGS, Q3 Q_NMOS_DGS, U1 Raspberry_Pi_2_3, U2 IC880A-SPI

Commit message: Re-add OSHW logo
Parts:
- added G***: LOGO, oshw-logos:OSHW_MASK_7MM, F.Cu at (136.4, 65.7)
Changed lines of the file:
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@@
     (links 45)
     (no_connects 0)
-    (area 100.889999 69.139999 189.940001 153.110001)
+    (area 49.911 40.259 162.941001 139.319001)
     (thickness 1.6)
     (drawings 9)
     (tracks 153)
     (zones 0)
-    (modules 14)
+    (modules 15)
     (nets 52)
   )
@@
     )
   )
+  (module oshw-logos:OSHW_MASK_7MM (layer F.Cu)
+    (at 136.435 65.725 270)
+    (fp_text reference G*** (at 0 3.71094 270) (layer F.Mask) hide
+      (effects (font (size 0.3175 0.3175) (thickness 0.0635)))
+    )
+    (fp_text value LOGO (at 0 -3.71094 270) (layer F.Mask) hide
+      (effects (font (size 0.3175 0.3175) (thickness 0.0635)))
+    )
+    (fp_poly (pts (xy -2.1209 3.14452) (xy -2.08534 3.1242) (xy -2.00152 3.0734) (xy -1.88468 2.9972)
+      (xy -1.74752 2.90322) (xy -1.60782 2.80924) (xy -1.49606 2.73304) (xy -1.41478 2.68224)
+      (xy -1.38176 2.66446) (xy -1.36398 2.66954) (xy -1.29794 2.70256) (xy -1.20142 2.75082)
+      (xy -1.14808 2.7813) (xy -1.05918 2.8194) (xy -1.016 2.82702) (xy -1.00838 2.81432)
+      (xy -0.97536 2.74574) (xy -0.92456 2.63144) (xy -0.85852 2.48158) (xy -0.78486 2.30378)
+      (xy -0.70358 2.11074) (xy -0.6223 1.91516) (xy -0.54356 1.72974) (xy -0.47498 1.5621)
+      (xy -0.42164 1.42494) (xy -0.38354 1.33096) (xy -0.37084 1.29032) (xy -0.37592 1.2827)
+      (xy -0.4191 1.23952) (xy -0.4953 1.1811) (xy -0.6604 1.04648) (xy -0.8255 0.84328)
+      (xy -0.92456 0.61214) (xy -0.95758 0.35306) (xy -0.92964 0.1143) (xy -0.83566 -0.1143)
+      (xy -0.67564 -0.32004) (xy -0.4826 -0.47244) (xy -0.254 -0.5715) (xy 0 -0.60198)
+      (xy 0.24384 -0.57404) (xy 0.47752 -0.4826) (xy 0.68326 -0.32512) (xy 0.77216 -0.22352)
+      (xy 0.89154 -0.01524) (xy 0.96012 0.20828) (xy 0.96774 0.26416) (xy 0.95758 0.51054)
+      (xy 0.88392 0.74676) (xy 0.75438 0.95758) (xy 0.57404 1.1303) (xy 0.55118 1.14554)
+      (xy 0.46736 1.20904) (xy 0.41148 1.25222) (xy 0.3683 1.28778) (xy 0.68072 2.03962)
+      (xy 0.73152 2.16154) (xy 0.81788 2.36728) (xy 0.89408 2.54508) (xy 0.9525 2.68478)
+      (xy 0.99568 2.77876) (xy 1.01346 2.81686) (xy 1.016 2.8194) (xy 1.04394 2.82448)
+      (xy 1.09982 2.80416) (xy 1.2065 2.75336) (xy 1.27508 2.7178) (xy 1.35636 2.67716)
+      (xy 1.39192 2.66446) (xy 1.4224 2.6797) (xy 1.4986 2.7305) (xy 1.61036 2.80416)
+      (xy 1.74498 2.8956) (xy 1.87452 2.9845) (xy 1.99136 3.0607) (xy 2.07772 3.11658)
+      (xy 2.11836 3.13944) (xy 2.12598 3.13944) (xy 2.16408 3.11912) (xy 2.23012 3.0607)
+      (xy 2.33426 2.96418) (xy 2.47904 2.82194) (xy 2.5019 2.79908) (xy 2.62128 2.67716)
+      (xy 2.7178 2.57556) (xy 2.7813 2.50444) (xy 2.8067 2.47142) (xy 2.8067 2.47142)
+      (xy 2.78384 2.43078) (xy 2.7305 2.34442) (xy 2.65176 2.22504) (xy 2.55524 2.08534)
+      (xy 2.30632 1.72212) (xy 2.44348 1.37922) (xy 2.48666 1.27508) (xy 2.54 1.14808)
+      (xy 2.5781 1.05664) (xy 2.59842 1.01854) (xy 2.63652 1.0033) (xy 2.7305 0.98298)
+      (xy 2.86512 0.95504) (xy 3.02768 0.92456) (xy 3.18262 0.89408) (xy 3.32232 0.86868)
+      (xy 3.42138 0.84836) (xy 3.4671 0.84074) (xy 3.47726 0.83312) (xy 3.48742 0.8128)
+      (xy 3.4925 0.76454) (xy 3.49758 0.68072) (xy 3.49758 0.5461) (xy 3.49758 0.35306)
+      (xy 3.49758 0.33274) (xy 3.49758 0.14732) (xy 3.4925 0.00254) (xy 3.48742 -0.09398)
+      (xy 3.48234 -0.13208) (xy 3.48234 -0.13208) (xy 3.43916 -0.14224) (xy 3.3401 -0.16256)
+      (xy 3.2004 -0.1905) (xy 3.0353 -0.22098) (xy 3.02514 -0.22352) (xy 2.8575 -0.25654)
+      (xy 2.72034 -0.28448) (xy 2.62382 -0.30734) (xy 2.58064 -0.32004) (xy 2.57302 -0.3302)
+      (xy 2.54 -0.39624) (xy 2.49174 -0.49784) (xy 2.4384 -0.62484) (xy 2.38252 -0.75438)
+      (xy 2.3368 -0.87122) (xy 2.30632 -0.95758) (xy 2.29616 -0.99822) (xy 2.29616 -0.99822)
+      (xy 2.32156 -1.03886) (xy 2.37744 -1.12268) (xy 2.45872 -1.24206) (xy 2.55524 -1.3843)
+      (xy 2.56286 -1.39446) (xy 2.65684 -1.53416) (xy 2.73558 -1.65354) (xy 2.78638 -1.73736)
+      (xy 2.8067 -1.77546) (xy 2.80416 -1.778) (xy 2.77368 -1.81864) (xy 2.70256 -1.89992)
+      (xy 2.60096 -2.0066) (xy 2.4765 -2.12852) (xy 2.4384 -2.16662) (xy 2.30378 -2.30124)
+      (xy 2.20726 -2.3876) (xy 2.14884 -2.43332) (xy 2.1209 -2.44348) (xy 2.1209 -2.44348)
+      (xy 2.07772 -2.41808) (xy 1.98882 -2.35966) (xy 1.86944 -2.27838) (xy 1.7272 -2.18186)
+      (xy 1.71704 -2.17678) (xy 1.57734 -2.08026) (xy 1.4605 -2.00152) (xy 1.37922 -1.94564)
+      (xy 1.34366 -1.92532) (xy 1.33604 -1.92532) (xy 1.28016 -1.94056) (xy 1.1811 -1.97612)
+      (xy 1.05664 -2.02438) (xy 0.9271 -2.07518) (xy 0.81026 -2.12598) (xy 0.72136 -2.16662)
+      (xy 0.68072 -2.18948) (xy 0.67818 -2.19202) (xy 0.66548 -2.24282) (xy 0.64008 -2.34696)
+      (xy 0.6096 -2.49174) (xy 0.57912 -2.66192) (xy 0.57404 -2.68986) (xy 0.54102 -2.85496)
+      (xy 0.51562 -2.99466) (xy 0.4953 -3.08864) (xy 0.48514 -3.12928) (xy 0.46228 -3.13436)
+      (xy 0.381 -3.13944) (xy 0.25654 -3.14198) (xy 0.10414 -3.14452) (xy -0.05334 -3.14452)
+      (xy -0.20828 -3.13944) (xy -0.34036 -3.13436) (xy -0.43434 -3.12928) (xy -0.47244 -3.12166)
+      (xy -0.47498 -3.11912) (xy -0.49022 -3.06832) (xy -0.51308 -2.96164) (xy -0.54102 -2.81686)
+      (xy -0.57404 -2.64668) (xy -0.57912 -2.6162) (xy -0.61214 -2.44856) (xy -0.64008 -2.3114)
+      (xy -0.6604 -2.21996) (xy -0.67056 -2.18186) (xy -0.6858 -2.17424) (xy -0.75438 -2.14376)
+      (xy -0.86614 -2.09804) (xy -1.0033 -2.04216) (xy -1.32334 -1.91262) (xy -1.71704 -2.18186)
+      (xy -1.7526 -2.20472) (xy -1.89484 -2.30124) (xy -2.00914 -2.37998) (xy -2.09042 -2.43078)
+      (xy -2.12344 -2.4511) (xy -2.12598 -2.44856) (xy -2.16662 -2.41554) (xy -2.24536 -2.34188)
+      (xy -2.3495 -2.23774) (xy -2.47396 -2.11582) (xy -2.5654 -2.02438) (xy -2.67462 -1.91262)
+      (xy -2.7432 -1.83896) (xy -2.77876 -1.7907) (xy -2.794 -1.76276) (xy -2.78892 -1.74498)
+      (xy -2.76352 -1.70434) (xy -2.70764 -1.61798) (xy -2.62636 -1.4986) (xy -2.52984 -1.3589)
+      (xy -2.4511 -1.24206) (xy -2.36728 -1.10998) (xy -2.3114 -1.016) (xy -2.29108 -0.97028)
+      (xy -2.29616 -0.9525) (xy -2.3241 -0.87376) (xy -2.36982 -0.75946) (xy -2.43078 -0.61976)
+      (xy -2.5654 -0.30988) (xy -2.77114 -0.26924) (xy -2.89306 -0.24638) (xy -3.06578 -0.21336)
+      (xy -3.23088 -0.18034) (xy -3.48996 -0.13208) (xy -3.50012 0.81534) (xy -3.45948 0.83312)
+      (xy -3.42138 0.84328) (xy -3.32486 0.8636) (xy -3.1877 0.89154) (xy -3.02768 0.92202)
+      (xy -2.89052 0.94742) (xy -2.75336 0.97536) (xy -2.6543 0.99314) (xy -2.60858 1.0033)
+      (xy -2.59842 1.01854) (xy -2.56286 1.08458) (xy -2.5146 1.19126) (xy -2.45872 1.31826)
+      (xy -2.40284 1.45288) (xy -2.35458 1.5748) (xy -2.32156 1.66878) (xy -2.30886 1.71704)
+      (xy -2.32664 1.7526) (xy -2.37998 1.83388) (xy -2.45618 1.95072) (xy -2.55016 2.08788)
+      (xy -2.64414 2.22504) (xy -2.72288 2.34188) (xy -2.77876 2.4257) (xy -2.80162 2.4638)
+      (xy -2.78892 2.49174) (xy -2.73558 2.55778) (xy -2.63144 2.66446) (xy -2.4765 2.81686)
+      (xy -2.4511 2.84226) (xy -2.32918 2.9591) (xy -2.22504 3.05562) (xy -2.15392 3.11912)
+      (xy -2.1209 3.14452)) (layer F.Mask) (width 0.00254))
+  )
   (gr_text "open source hardware" (at 136.271 83.439 270) (layer F.Mask)

Commit message: Add SHT21 sensor
Parts:
- added C1: C, Capacitors_SMD:C_1206_HandSoldering, F.Cu at (149.4, 103.2)
- added U3: SHT21, sensirion:SHT21, F.Cu at (143.4, 103.2)
- J1: value I2C -> I2C_HEADER
- J3: value SER -> SERIAL_HEADER
- J4: value PWR -> PWR_HEADER
Routing:
- net /3.3V: track 195.6 -> 240.1 mm, vias 0 -> 2
- net GND: track 13.4 -> 33.1 mm
- net Net-(J1-Pad2): track 99.7 -> 119.2 mm, vias 1 -> 2
- net Net-(J1-Pad1): track 101.4 -> 116.2 mm, vias 1 -> 2
Other:
- outline, holes or cut-outs redrawn

Commit message: Add Raspberry Pi mounting holes
Parts:
- added REF**: MountingHole_2.7mm_M2.5, Mounting_Holes:MountingHole_2.7mm_M2.5, F.Cu at (140.3, 79.3)
- added REF**: MountingHole_2.7mm_M2.5, Mounting_Holes:MountingHole_2.7mm_M2.5, F.Cu at (82.3, 79.3)
- added REF**: MountingHole_2.7mm_M2.5, Mounting_Holes:MountingHole_2.7mm_M2.5, F.Cu at (140.3, 128.3)
- added REF**: MountingHole_2.7mm_M2.5, Mounting_Holes:MountingHole_2.7mm_M2.5, F.Cu at (82.3, 128.3)
- C1: footprint Capacitors_SMD:C_1206_HandSoldering -> Capacitors_SMD:C_1206
- J3: value SERIAL_HEADER -> SER
- J4: value PWR_HEADER -> PWR
- moved J3 78.5 mm to (71.2, 124.7)
- moved J4 5.68 mm to (148.9, 129.5)
- moved G*** 2.50 mm to (136.4, 68.2)
Routing:
- net Net-(J3-Pad1): track 27.6 -> 60.6 mm, vias 0 -> 1
- net Net-(J3-Pad2): track 28.2 -> 57.6 mm, vias 0 -> 1
- net /5V: track 215.7 -> 229.3 mm
- net GND: track 33.1 -> 25.8 mm
- net Net-(U1-Pad22): track 66.1 -> 72.9 mm
- net Net-(U1-Pad24): track 86.6 -> 93.1 mm
- net Net-(Q3-Pad2): track 22.1 -> 27.6 mm
- net (no net): track 4.57 -> 0.00 mm
- net Net-(Q2-Pad2): track 51.6 -> 54.5 mm
- net Net-(J1-Pad2): track 119.2 -> 121.8 mm
- net Net-(Q1-Pad2): track 67.2 -> 68.4 mm
- net Net-(J1-Pad1): track 116.2 -> 117.1 mm
Other:
- board text added: "5V"
- board text added: "GND"
- board text added: "OSHW"
- board text added: "RX"
- board text added: "TX"
- board text removed: "open source hardware"

Commit message: Nicer keepout area around sensor
Routing:
- net GND: track 25.8 -> 30.4 mm
Changed lines of the file:
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@@
     (thickness 1.6)
     (drawings 30)
-    (tracks 200)
+    (tracks 201)
     (zones 0)
     (modules 21)
@@
   )
   (setup
-    (last_trace_width 0.25)
+    (last_trace_width 0.4)
     (user_trace_width 0.4)
     (trace_clearance 0.2)
@@
   (segment (start 88.61341 131.225) (end 90.517 131.225) (width 0.25) (layer F.Cu) (net 11))
   (segment (start 90.517 131.225) (end 92.202 129.54) (width 0.25) (layer F.Cu) (net 11))
+  (segment (start 138.049 105.029) (end 138.049 109.614) (width 0.4) (layer F.Cu) (net 12))
   (segment (start 143.435 106.963) (end 140.941 106.963) (width 0.4) (layer F.Cu) (net 12))
   (segment (start 140.941 106.963) (end 140.843 106.865) (width 0.4) (layer F.Cu) (net 12))
@@
       )
     )
+  )
+  (zone (net 0) (net_name "") (layer F.Cu) (hatch edge 0.508)
+    (connect_pads (clearance 0.381))
+    (min_thickness 0.254)
+    (keepout (tracks allowed) (vias allowed) (copperpour not_allowed))
+    (fill yes (arc_segments 16) (thermal_gap 0.508) (thermal_bridge_width 0.508))
+    (polygon
+      (pts
+        (xy 139.16 109.425) (xy 137.185 109.425) (xy 134.885 107.25) (xy 135.835 104.925) (xy 137.66 103.875)
+        (xy 138.91 104.025) (xy 138.66 109) (xy 139.335 109.15)
+      )
+    )
