File: backplane.kicad_pcb (KiCad board)
At the start: 2 copper layers, 88.9 x 83.8 mm, 33 parts, among them J1 I2C, J2 I2C, J3 SER, J4 PWR, J5 FAN, Q1 Q_NMOS_DGS, Q2 Q_NMOS_DGS, Q3 Q_NMOS_DGS, Q4 Q_NMOS_DGS, U1 Raspberry_Pi_2_3, U2 IC880A-SPI, U3 SHT21

Commit message: Switch PWM pin for fan
Connections:
- U1 pad 12: Net-(U1-Pad12) -> Net-(Q4-Pad2)
- U1 pad 35: Net-(Q4-Pad2) -> Net-(U1-Pad35)
Routing:
- net Net-(Q4-Pad2): track 78.8 -> 114.0 mm, vias 3 -> 6
- net GND: track 30.4 -> 24.4 mm
- net Net-(U1-Pad29): track 12.0 -> 13.9 mm

Commit message: Small changes
Other:
- board text added: "+"
Changed lines of the file:
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@@
     (area 63.805999 51.613999 152.856001 135.584001)
     (thickness 1.6)
-    (drawings 83)
+    (drawings 86)
     (tracks 288)
     (zones 0)
@@
     )
   )
+  (gr_text + (at 70.885 109.7) (layer F.SilkS)
+    (effects (font (size 0.8 0.8) (thickness 0.15)))
+  )
+  (gr_text + (at 70.86 99.525) (layer F.SilkS)
+    (effects (font (size 0.8 0.8) (thickness 0.15)))
+  )
+  (gr_text + (at 70.86 89.375) (layer F.SilkS)
+    (effects (font (size 0.8 0.8) (thickness 0.15)))
+  )
   (gr_text 5V (at 76.935 58.225) (layer F.SilkS)

Commit message: Add Github URL to back side
Other:
- board text added: "https://github.com/dbrgn/ic880a-backplane"
Changed lines of the file:
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@@
     (area 63.805999 51.613999 152.856001 135.584001)
     (thickness 1.6)
-    (drawings 86)
+    (drawings 87)
     (tracks 288)
     (zones 0)
@@
     )
   )
+  (gr_text https://github.com/dbrgn/ic880a-backplane (at 120.435 61.225) (layer B.SilkS)
+    (effects (font (size 1.5 1.5) (thickness 0.3)) (justify mirror))
+  )
   (gr_text + (at 70.885 109.7) (layer F.SilkS)

Commit message: Start integrating MP1584 dc converter board
Parts:
- added J5: PWR, Connectors_Terminal_Blocks:TerminalBlock_Pheonix_MPT-2.54mm_2pol, F.Cu at (72.3, 132.1)
- added U4: MP1584_MODULE, regulators:MP1584_MODULE, F.Cu at (125.7, 68.2)
- renumbered J5 to J6
Routing:
- net Net-(Q2-Pad2): track 49.1 -> 48.3 mm
- net Net-(Q1-Pad2): track 63.0 -> 62.3 mm
- net Net-(Q3-Pad2): track 26.7 -> 26.0 mm

Commit message: Use screw terminal for PWR
Parts:
- J4: footprint headers:header_1x2_marked -> Connectors_Terminal_Blocks:TerminalBlock_Pheonix_MPT-2.54mm_2pol
- moved J4 4.96 mm to (149.5, 126.7), turned to 90 degrees
Routing:
- net /5V: track 276.4 -> 271.9 mm
Other:
- board text added: "PWR (5V)"
Changed lines of the file:
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@@
   (general
     (links 75)
-    (no_connects 7)
+    (no_connects 9)
     (area 63.805999 51.613999 152.856001 135.584001)
     (thickness 1.6)
-    (drawings 87)
-    (tracks 289)
+    (drawings 88)
+    (tracks 286)
     (zones 0)
     (modules 35)
@@
     )
   )
-  (module headers:header_1x2_marked (layer F.Cu)
-    (at 144.935 128.515 180)
-    (descr "Through hole straight pin header, 1x02, 2.54mm pitch, single row")
-    (tags "Through hole pin header THT 1x02 2.54mm single row")
-    (fp_text reference J4 (at 0.0275 4.953 180) (layer F.SilkS) hide
-      (effects (font (size 1 1) (thickness 0.15)))
-    )
-    (fp_text value PWR (at 0.0275 -2.54 180) (layer F.SilkS)
-      (effects (font (size 1 1) (thickness 0.15)))
-    )
-    (fp_line (start -1.27 3.81) (end -1.27 -1.27) (layer F.SilkS) (width 0.2))
-    (fp_line (start 1.27 3.81) (end -1.27 3.81) (layer F.SilkS) (width 0.2))
-    (fp_line (start 1.27 -1.27) (end 1.27 3.81) (layer F.SilkS) (width 0.2))
-    (fp_line (start -1.27 -1.27) (end 1.27 -1.27) (layer F.SilkS) (width 0.2))
-    (fp_line (start -1.27 -1.27) (end -1.27 3.81) (layer F.Fab) (width 0.1))
-    (fp_line (start -1.27 3.81) (end 1.27 3.81) (layer F.Fab) (width 0.1))
-    (fp_line (start 1.27 3.81) (end 1.27 -1.27) (layer F.Fab) (width 0.1))
-    (fp_line (start 1.27 -1.27) (end -1.27 -1.27) (layer F.Fab) (width 0.1))
-    (fp_line (start -1.6 -1.6) (end -1.6 4.1) (layer F.CrtYd) (width 0.05))
-    (fp_line (start -1.6 4.1) (end 1.6 4.1) (layer F.CrtYd) (width 0.05))
-    (fp_line (start 1.6 4.1) (end 1.6 -1.6) (layer F.CrtYd) (width 0.05))
-    (fp_line (start 1.6 -1.6) (end -1.6 -1.6) (layer F.CrtYd) (width 0.05))
-    (pad 1 thru_hole rect (at 0 0 180) (size 1.7 1.7) (drill 1) (layers *.Cu *.Mask)
-      (net 12 GND))
-    (pad 2 thru_hole oval (at 0 2.54 180) (size 1.7 1.7) (drill 1) (layers *.Cu *.Mask)
-      (net 45 /5V))
-    (model Socket_Strips.3dshapes/Socket_Strip_Straight_1x02.wrl
-      (at (xyz 0 -0.05 0))
-      (scale (xyz 1 1 1))
-      (rotate (xyz 0 0 90))
-    )
-  )
   (module Mounting_Holes:MountingHole_2.7mm_M2.5 (layer F.Cu)
     (at 149.185 131.975)
@@
     )
   )
+  (module Connectors_Terminal_Blocks:TerminalBlock_Pheonix_MPT-2.54mm_2pol (layer F.Cu)
+    (at 149.535 126.665 90)
+    (descr "2-way 2.54mm pitch terminal block, Phoenix MPT series")
+    (fp_text reference J4 (at 3.5 -4.1 90) (layer F.SilkS) hide
+      (effects (font (size 1 1) (thickness 0.15)))
+    )
+    (fp_text value PWR (at 1.27 4.50088 90) (layer F.Fab) hide
+      (effects (font (size 1 1) (thickness 0.15)))
+    )
+    (fp_line (start -1.7 -3.3) (end 4.3 -3.3) (layer F.CrtYd) (width 0.05))
+    (fp_line (start -1.7 3.3) (end -1.7 -3.3) (layer F.CrtYd) (width 0.05))
+    (fp_line (start 4.3 3.3) (end -1.7 3.3) (layer F.CrtYd) (width 0.05))
+    (fp_line (start 4.3 -3.3) (end 4.3 3.3) (layer F.CrtYd) (width 0.05))
+    (fp_line (start 4.06908 2.60096) (end -1.52908 2.60096) (layer F.SilkS) (width 0.15))
+    (fp_line (start -1.33096 3.0988) (end -1.33096 2.60096) (layer F.SilkS) (width 0.15))
+    (fp_line (start 3.87096 2.60096) (end 3.87096 3.0988) (layer F.SilkS) (width 0.15))
+    (fp_line (start 1.27 3.0988) (end 1.27 2.60096) (layer F.SilkS) (width 0.15))
+    (fp_line (start -1.52908 -2.70002) (end 4.06908 -2.70002) (layer F.SilkS) (width 0.15))
+    (fp_line (start -1.52908 3.0988) (end 4.06908 3.0988) (layer F.SilkS) (width 0.15))
+    (fp_line (start 4.06908 3.0988) (end 4.06908 -3.0988) (layer F.SilkS) (width 0.15))
+    (fp_line (start 4.06908 -3.0988) (end -1.52908 -3.0988) (layer F.SilkS) (width 0.15))
+    (fp_line (start -1.52908 -3.0988) (end -1.52908 3.0988) (layer F.SilkS) (width 0.15))
+    (pad 2 thru_hole oval (at 2.54 0 90) (size 1.99898 1.99898) (drill 1.09728) (layers *.Cu *.Mask)
+      (net 45 /5V))
+    (pad 1 thru_hole rect (at 0 0 90) (size 1.99898 1.99898) (drill 1.09728) (layers *.Cu *.Mask)
+      (net 12 GND))
+    (model Terminal_Blocks.3dshapes/TerminalBlock_Pheonix_MPT-2.54mm_2pol.wrl
+      (at (xyz 0.05 0 0))
+      (scale (xyz 1 1 1))
+      (rotate (xyz 0 0 0))
+    )
+  )
+  (gr_text "PWR (5V)" (at 145.335 125.325 90) (layer F.SilkS)
+    (effects (font (size 0.8 0.8) (thickness 0.15)))
+  )
   (gr_text https://github.com/dbrgn/ic880a-backplane (at 120.435 61.225) (layer B.SilkS)
     (effects (font (size 1.5 1.5) (thickness 0.3)) (justify mirror))
@@
     (effects (font (size 0.8 0.8) (thickness 0.15)) (justify left))
   )
-  (gr_text 5V (at 146.935 125.975) (layer F.SilkS)
-    (effects (font (size 0.8 0.8) (thickness 0.15)) (justify left))
-  )
-  (gr_text GND (at 146.935 128.515) (layer F.SilkS)
-    (effects (font (size 0.8 0.8) (thickness 0.15)) (justify left))
+  (gr_text 5V (at 149.535 121.825) (layer F.SilkS)
+    (effects (font (size 0.8 0.8) (thickness 0.15)))
+  )
+  (gr_text GND (at 149.535 128.925) (layer F.SilkS)
+    (effects (font (size 0.8 0.8) (thickness 0.15)))
   )
   (gr_text iC880A-SPI (at 150.035 114.825 90) (layer F.SilkS)
@@
   (segment (start 133.135 86.325) (end 133.135 85.425) (width 0.4) (layer F.Cu) (net 44))
   (segment (start 133.135 85.425) (end 131.985 84.275) (width 0.4) (layer F.Cu) (net 44))
+  (segment (start 143.435 133.225) (end 145.435 131.225) (width 0.8) (layer B.Cu) (net 45))
+  (segment (start 145.435 131.225) (end 145.435 126.975) (width 0.8) (layer B.Cu) (net 45))
+  (segment (start 145.435 126.975) (end 148.285 124.125) (width 0.8) (layer B.Cu) (net 45))
+  (segment (start 148.285 124.125) (end 149.535 124.125) (width 0.8) (layer B.Cu) (net 45))
   (segment (start 131.699 132.334) (end 130.058 133.975) (width 0.8) (layer B.Cu) (net 45))
   (segment (start 130.058 133.975) (end 80.885 133.975) (width 0.8) (layer B.Cu) (net 45))
@@
   (segment (start 64.685 74.175) (end 66.435 72.425) (width 0.8) (layer B.Cu) (net 45))
   (segment (start 64.685 89.715) (end 66.421 87.979) (width 0.8) (layer B.Cu) (net 45))
-  (segment (start 144.935 125.975) (end 146.137081 125.975) (width 0.8) (layer B.Cu) (net 45))
-  (segment (start 143.934999 132.725001) (end 143.435 133.225) (width 0.8) (layer B.Cu) (net 45))
-  (segment (start 146.137081 125.975) (end 146.935 126.772919) (width 0.8) (layer B.Cu) (net 45))
-  (segment (start 146.935 126.772919) (end 146.935 129.725) (width 0.8) (layer B.Cu) (net 45))
-  (segment (start 146.935 129.725) (end 143.934999 132.725001) (width 0.8) (layer B.Cu) (net 45))
   (segment (start 135.382 129.54) (end 137.817 131.975) (width 0.8) (layer F.Cu) (net 45))
   (segment (start 137.817 131.975) (end 141.477894 131.975) (width 0.8) (layer F.Cu) (net 45))
@@
   (segment (start 89.535 64.135) (end 144.935 119.535) (width 0.8) (layer F.Cu) (net 45))
   (segment (start 89.535 56.9097) (end 89.535 64.135) (width 0.8) (layer F.Cu) (net 45))
-  (segment (start 144.935 119.535) (end 144.935 125.975) (width 0.8) (layer F.Cu) (net 45))
-  (segment (start 144.694998 125.975) (end 144.935 125.975) (width 0.8) (layer F.Cu) (net 45))
   (segment (start 132.842 129.54) (end 132.842 131.064) (width 0.8) (layer F.Cu) (net 45))
   (segment (start 132.842 131.064) (end 131.699 132.334) (width 0.8) (layer F.Cu) (net 45))

Commit message: Improvements
Parts:
- moved J3 13.9 mm to (75.3, 132.4), turned to 270 degrees
- moved J5 10.0 mm to (67.1, 123.5), turned to 270 degrees
Routing:
- net Net-(J3-Pad1): track 67.4 -> 48.9 mm
- net Net-(J3-Pad2): track 63.7 -> 45.7 mm
- net /5V: track 271.9 -> 267.5 mm
Other:
- board text added: "6.7-28V"
- board text added: "PWR (Conv)"
- board text added: "PWR (Direct)"
- board text removed: "PWR (5V)"
Changed lines of the file:
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@@
     (area 63.805999 51.613999 152.856001 135.584001)
     (thickness 1.6)
-    (drawings 88)
-    (tracks 286)
+    (drawings 91)
+    (tracks 282)
     (zones 0)
     (modules 35)
@@
   )
   (module headers:header_1x2_unmarked (layer F.Cu)
-    (at 66.421 121.685)
+    (at 75.334807 132.375117 270)
     (descr "Through hole straight pin header, 1x02, 2.54mm pitch, single row")
     (tags "Through hole pin header THT 1x02 2.54mm single row")
-    (fp_text reference J3 (at -0.0015 -2.4475) (layer F.SilkS) hide
-      (effects (font (size 1 1) (thickness 0.15)))
-    )
-    (fp_text value SER (at -0.0015 5.0455) (layer F.SilkS)
+    (fp_text reference J3 (at -0.0015 -2.4475 270) (layer F.SilkS) hide
+      (effects (font (size 1 1) (thickness 0.15)))
+    )
+    (fp_text value SER (at -2.250117 2.299807 360) (layer F.SilkS)
       (effects (font (size 1 1) (thickness 0.15)))
     )
@@
     (fp_line (start 1.6 4.1) (end 1.6 -1.6) (layer F.CrtYd) (width 0.05))
     (fp_line (start 1.6 -1.6) (end -1.6 -1.6) (layer F.CrtYd) (width 0.05))
-    (pad 1 thru_hole circle (at 0 0) (size 1.7 1.7) (drill 1) (layers *.Cu *.Mask)
+    (pad 1 thru_hole circle (at 0 0 270) (size 1.7 1.7) (drill 1) (layers *.Cu *.Mask)
       (net 9 "Net-(J3-Pad1)"))
-    (pad 2 thru_hole oval (at 0 2.54) (size 1.7 1.7) (drill 1) (layers *.Cu *.Mask)
+    (pad 2 thru_hole oval (at 0 2.54 270) (size 1.7 1.7) (drill 1) (layers *.Cu *.Mask)
       (net 10 "Net-(J3-Pad2)"))
     (model Socket_Strips.3dshapes/Socket_Strip_Straight_1x02.wrl
@@
   (module regulators:MP1584_MODULE (layer F.Cu)
     (at 125.706 68.161 180)
-    (fp_text reference U4 (at 0 9.652 180) (layer F.SilkS)
+    (fp_text reference U4 (at 0 9.652 180) (layer F.SilkS) hide
       (effects (font (size 1 1) (thickness 0.15)))
     )
@@
   )
   (module Connectors_Terminal_Blocks:TerminalBlock_Pheonix_MPT-2.54mm_2pol (layer F.Cu)
-    (at 72.335 132.125)
+    (at 67.135 123.525 270)
     (descr "2-way 2.54mm pitch terminal block, Phoenix MPT series")
-    (fp_text reference J5 (at -0.5 -4.1) (layer F.SilkS)
-      (effects (font (size 1 1) (thickness 0.15)))
-    )
-    (fp_text value PWR (at 5.1 -0.1 270) (layer F.SilkS)
+    (fp_text reference J5 (at 3.8 -5.4 360) (layer F.SilkS) hide
+      (effects (font (size 1 1) (thickness 0.15)))
+    )
+    (fp_text value PWR (at 2.2 -3.9 270) (layer F.SilkS) hide
       (effects (font (size 1 1) (thickness 0.15)))
     )
@@
     (fp_line (start 4.06908 -3.0988) (end -1.52908 -3.0988) (layer F.SilkS) (width 0.15))
     (fp_line (start -1.52908 -3.0988) (end -1.52908 3.0988) (layer F.SilkS) (width 0.15))
-    (pad 2 thru_hole oval (at 2.54 0) (size 1.99898 1.99898) (drill 1.09728) (layers *.Cu *.Mask)
+    (pad 2 thru_hole oval (at 2.54 0 270) (size 1.99898 1.99898) (drill 1.09728) (layers *.Cu *.Mask)
       (net 56 "Net-(J5-Pad2)"))
-    (pad 1 thru_hole rect (at 0 0) (size 1.99898 1.99898) (drill 1.09728) (layers *.Cu *.Mask)
+    (pad 1 thru_hole rect (at 0 0 270) (size 1.99898 1.99898) (drill 1.09728) (layers *.Cu *.Mask)
       (net 55 "Net-(J5-Pad1)"))
     (model Terminal_Blocks.3dshapes/TerminalBlock_Pheonix_MPT-2.54mm_2pol.wrl
@@
     )
   )
-  (gr_text "PWR (5V)" (at 145.335 125.325 90) (layer F.SilkS)
+  (gr_text "PWR\n(Conv)" (at 71.835 124.925 90) (layer F.SilkS)
+    (effects (font (size 0.8 0.8) (thickness 0.15)))
+  )
+  (gr_text 6.7-28V (at 64.535 128.425) (layer F.SilkS)
+    (effects (font (size 0.8 0.8) (thickness 0.15)) (justify left))
+  )
+  (gr_text GND (at 64.535 121.325) (layer F.SilkS)
+    (effects (font (size 0.8 0.8) (thickness 0.15)) (justify left))
+  )
+  (gr_text "PWR\n(Direct)" (at 144.635 125.325 90) (layer F.SilkS)
     (effects (font (size 0.8 0.8) (thickness 0.15)))
   )
@@
     (effects (font (size 0.8 0.8) (thickness 0.15)) (justify left))
   )
-  (gr_text 5V (at 149.535 121.825) (layer F.SilkS)
-    (effects (font (size 0.8 0.8) (thickness 0.15)))
-  )
-  (gr_text GND (at 149.535 128.925) (layer F.SilkS)
-    (effects (font (size 0.8 0.8) (thickness 0.15)))
+  (gr_text 5V (at 152.135 121.825) (layer F.SilkS)
+    (effects (font (size 0.8 0.8) (thickness 0.15)) (justify right))
+  )
+  (gr_text GND (at 152.135 128.925) (layer F.SilkS)
+    (effects (font (size 0.8 0.8) (thickness 0.15)) (justify right))
   )
   (gr_text iC880A-SPI (at 150.035 114.825 90) (layer F.SilkS)
@@
     (effects (font (size 0.8 0.8) (thickness 0.15)) (justify left))
   )
-  (gr_text RX (at 68.453 124.225) (layer F.SilkS)
-    (effects (font (size 0.8 0.8) (thickness 0.15)) (justify left))
-  )
-  (gr_text TX (at 68.453 121.725) (layer F.SilkS)
-    (effects (font (size 0.8 0.8) (thickness 0.15)) (justify left))
+  (gr_text RX (at 72.794807 134.407117) (layer F.SilkS)
+    (effects (font (size 0.8 0.8) (thickness 0.15)))
+  )
+  (gr_text TX (at 75.294807 134.407117) (layer F.SilkS)
+    (effects (font (size 0.8 0.8) (thickness 0.15)))
   )
   (gr_line (start 139.265 89.719) (end 139.265 86.163) (angle 90) (layer Edge.Cuts) (width 0.15))
@@
   (segment (start 136.135 89.325) (end 136.135 90.225) (width 0.4) (layer F.Cu) (net 8))
   (segment (start 136.135 90.225) (end 136.7758 90.8658) (width 0.4) (layer F.Cu) (net 8))
-  (segment (start 66.435 121.725) (end 70.435 121.725) (width 0.25) (layer B.Cu) (net 9))
   (segment (start 126.119315 131.975) (end 126.685 131.975) (width 0.25) (layer B.Cu) (net 9))
-  (segment (start 70.435 121.725) (end 80.685 131.975) (width 0.25) (layer B.Cu) (net 9))
   (segment (start 80.685 131.975) (end 126.119315 131.975) (width 0.25) (layer B.Cu) (net 9))
   (segment (start 127.084999 131.575001) (end 126.685 131.975) (width 0.25) (layer F.Cu) (net 9))
@@
   (segment (start 127.762 130.898) (end 127.084999 131.575001) (width 0.25) (layer F.Cu) (net 9))
   (via (at 126.685 131.975) (size 0.8) (drill 0.6) (layers F.Cu B.Cu) (net 9))
-  (segment (start 66.435 124.225) (end 72.235 124.225) (width 0.25) (layer B.Cu) (net 10))
-  (segment (start 72.235 124.225) (end 80.835 132.825) (width 0.25) (layer B.Cu) (net 10))
   (segment (start 80.835 132.825) (end 120.869315 132.825) (width 0.25) (layer B.Cu) (net 10))
   (segment (start 120.869315 132.825) (end 121.435 132.825) (width 0.25) (layer B.Cu) (net 10))
@@
   (segment (start 133.135 86.325) (end 133.135 85.425) (width 0.4) (layer F.Cu) (net 44))
   (segment (start 133.135 85.425) (end 131.985 84.275) (width 0.4) (layer F.Cu) (net 44))
+  (segment (start 131.699 132.334) (end 130.058 133.975) (width 0.8) (layer B.Cu) (net 45))
+  (segment (start 130.058 133.975) (end 80.885 133.975) (width 0.8) (layer B.Cu) (net 45))
+  (segment (start 64.685 116.475) (end 64.685 89.715) (width 0.8) (layer B.Cu) (net 45))
+  (segment (start 80.885 133.975) (end 73.135 126.225) (width 0.8) (layer B.Cu) (net 45))
+  (segment (start 73.135 124.925) (end 64.685 116.475) (width 0.8) (layer B.Cu) (net 45))
+  (segment (start 73.135 126.225) (end 73.135 124.925) (width 0.8) (layer B.Cu) (net 45))
   (segment (start 143.435 133.225) (end 145.435 131.225) (width 0.8) (layer B.Cu) (net 45))
   (segment (start 145.435 131.225) (end 145.435 126.975) (width 0.8) (layer B.Cu) (net 45))
   (segment (start 145.435 126.975) (end 148.285 124.125) (width 0.8) (layer B.Cu) (net 45))
   (segment (start 148.285 124.125) (end 149.535 124.125) (width 0.8) (layer B.Cu) (net 45))
-  (segment (start 131.699 132.334) (end 130.058 133.975) (width 0.8) (layer B.Cu) (net 45))
-  (segment (start 130.058 133.975) (end 80.885 133.975) (width 0.8) (layer B.Cu) (net 45))
-  (segment (start 80.885 133.975) (end 73.135 126.225) (width 0.8) (layer B.Cu) (net 45))
-  (segment (start 65.685 126.225) (end 64.685 125.225) (width 0.8) (layer B.Cu) (net 45))
-  (segment (start 73.135 126.225) (end 65.685 126.225) (width 0.8) (layer B.Cu) (net 45))
-  (segment (start 64.685 125.225) (end 64.685 89.715) (width 0.8) (layer B.Cu) (net 45))
   (segment (start 76.435 68.225) (end 74.835 68.225) (width 0.8) (layer F.Cu) (net 45))
   (segment (start 76.435 68.225) (end 85.445 68.225) (width 0.8) (layer F.Cu) (net 45))

Commit message: Change annotation of LED MOSFETs
Parts:
- renumbered Q3 to Q1, Q1 to Q3
Connections:
- Q1 pad 1: Net-(D1-Pad1) -> Net-(D3-Pad1)
- Q3 pad 1: Net-(D3-Pad1) -> Net-(D1-Pad1)
- U1 pad 36: Net-(Q1-Pad2) -> Net-(Q3-Pad2)
- U1 pad 40: Net-(Q3-Pad2) -> Net-(Q1-Pad2)
Routing:
- net Net-(Q3-Pad2): track 26.0 -> 11.9 mm
- net Net-(Q1-Pad2): track 62.3 -> 76.4 mm
Changed lines of the file:
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@@
   (general
     (links 75)
-    (no_connects 9)
+    (no_connects 14)
     (area 63.805999 51.613999 152.856001 135.584001)
     (thickness 1.6)
@@
       (net 54 "Net-(U1-Pad35)"))
     (pad 36 thru_hole oval (at 2.54 43.18 270) (size 1.7 1.7) (drill 1) (layers *.Cu *.Mask)
-      (net 11 "Net-(Q1-Pad2)"))
+      (net 14 "Net-(Q3-Pad2)"))
     (pad 37 thru_hole oval (at 0 45.72 270) (size 1.7 1.7) (drill 1) (layers *.Cu *.Mask)
       (net 33 "Net-(U1-Pad37)"))
@@
       (net 12 GND))
     (pad 40 thru_hole oval (at 2.54 48.26 270) (size 1.7 1.7) (drill 1) (layers *.Cu *.Mask)
-      (net 14 "Net-(Q3-Pad2)"))
+      (net 11 "Net-(Q1-Pad2)"))
     (model Pin_Headers.3dshapes/Pin_Header_Straight_2x20.wrl
       (at (xyz 0.05 -0.95 -0.2))
@@
     (tags SOT-23)
     (attr smd)
-    (fp_text reference Q1 (at 0 -2.5) (layer F.SilkS)
+    (fp_text reference Q3 (at 0 -2.5) (layer F.SilkS)
       (effects (font (size 1 1) (thickness 0.15)))
     )
@@
     (fp_line (start 0.76 1.58) (end -0.7 1.58) (layer F.SilkS) (width 0.12))
     (pad 1 smd rect (at -1.5 -0.95) (size 1.9 0.8) (layers F.Cu F.Paste F.Mask)
-      (net 6 "Net-(D3-Pad1)"))
+      (net 2 "Net-(D1-Pad1)"))
     (pad 2 smd rect (at -1.5 0.95) (size 1.9 0.8) (layers F.Cu F.Paste F.Mask)
       (net 11 "Net-(Q1-Pad2)"))
@@
     (tags SOT-23)
     (attr smd)
-    (fp_text reference Q3 (at 0 -2.5) (layer F.SilkS)
+    (fp_text reference Q1 (at 0 -2.5) (layer F.SilkS)
       (effects (font (size 1 1) (thickness 0.15)))
     )
@@
     (fp_line (start 0.76 1.58) (end -0.7 1.58) (layer F.SilkS) (width 0.12))
     (pad 1 smd rect (at -1.5 -0.95) (size 1.9 0.8) (layers F.Cu F.Paste F.Mask)
-      (net 2 "Net-(D1-Pad1)"))
+      (net 6 "Net-(D3-Pad1)"))
     (pad 2 smd rect (at -1.5 0.95) (size 1.9 0.8) (layers F.Cu F.Paste F.Mask)
       (net 14 "Net-(Q3-Pad2)"))
@@
   (segment (start 70.551 95.819) (end 65.935 100.435) (width 0.25) (layer F.Cu) (net 11))
   (segment (start 73.935 124.225) (end 73.935 125.925) (width 0.25) (layer F.Cu) (net 11))
-  (segment (start 87.11341 132.725) (end 88.61341 131.225) (width 0.25) (layer F.Cu) (net 11))
-  (segment (start 88.61341 131.225) (end 90.517 131.225) (width 0.25) (layer F.Cu) (net 11))
   (segment (start 65.935 100.435) (end 65.935 116.225) (width 0.25) (layer F.Cu) (net 11))
   (segment (start 65.935 116.225) (end 73.935 124.225) (width 0.25) (layer F.Cu) (net 11))
   (segment (start 73.935 125.925) (end 80.735 132.725) (width 0.25) (layer F.Cu) (net 11))
   (segment (start 80.735 132.725) (end 87.11341 132.725) (width 0.25) (layer F.Cu) (net 11))
-  (segment (start 90.517 131.225) (end 92.202 129.54) (width 0.25) (layer F.Cu) (net 11))
+  (segment (start 87.122 129.54) (end 87.122 131.288) (width 0.25) (layer F.Cu) (net 11))
+  (segment (start 87.122 131.288) (end 86.685 131.725) (width 0.25) (layer F.Cu) (net 11))
+  (segment (start 86.685 131.725) (end 81.135 131.725) (width 0.25) (layer F.Cu) (net 11))
+  (segment (start 81.135 131.725) (end 75.081 125.671) (width 0.25) (layer F.Cu) (net 11))
+  (segment (start 87.11341 132.725) (end 88.61341 131.225) (width 0.25) (layer F.Cu) (net 11))
+  (segment (start 88.61341 131.225) (end 90.517 131.225) (width 0.25) (layer F.Cu) (net 11))
   (segment (start 138.249 93.529) (end 138.249 98.114) (width 0.4) (layer F.Cu) (net 12))
   (segment (start 143.635 95.463) (end 141.141 95.463) (width 0.4) (layer F.Cu) (net 12))
@@
   (segment (start 88.812001 130.389999) (end 89.662 129.54) (width 0.25) (layer F.Cu) (net 13))
   (segment (start 86.977 132.225) (end 88.812001 130.389999) (width 0.25) (layer F.Cu) (net 13))
-  (segment (start 87.122 129.54) (end 87.122 131.288) (width 0.25) (layer F.Cu) (net 14))
-  (segment (start 87.122 131.288) (end 86.685 131.725) (width 0.25) (layer F.Cu) (net 14))
-  (segment (start 86.685 131.725) (end 81.135 131.725) (width 0.25) (layer F.Cu) (net 14))
-  (segment (start 81.135 131.725) (end 75.081 125.671) (width 0.25) (layer F.Cu) (net 14))
+  (segment (start 90.517 131.225) (end 92.202 129.54) (width 0.25) (layer F.Cu) (net 14))
   (segment (start 75.081 125.671) (end 75.081 116.139) (width 0.25) (layer F.Cu) (net 14))
   (segment (start 125.2171 118.1276) (end 125.2171 121.1531) (width 0.25) (layer F.Cu) (net 21) (status 10))
