File: backplane.kicad_pcb (KiCad board)
At the start: 2 copper layers, 88.9 x 83.8 mm, 35 parts, among them J1 I2C, J2 I2C, J3 SER, J4 PWR, J5 PWR, J6 FAN, Q1 Q_NMOS_DGS, Q2 Q_NMOS_DGS, Q3 Q_NMOS_DGS, Q4 Q_NMOS_DGS, U1 Raspberry_Pi_2_3, U2 IC880A-SPI, U3 SHT21, U4 MP1584_MODULE

Commit message: Move LEDs closer together
Parts:
- moved D1 2.40 mm to (69.6, 110.2)
- moved D3 2.40 mm to (69.6, 94.7)
- moved Q3 2.40 mm to (76.6, 97.3)
- moved Q1 2.40 mm to (76.6, 112.8)
Connections:
- Q1 pad 1: Net-(D3-Pad1) -> Net-(D1-Pad1)
- Q1 pad 2: Net-(Q3-Pad2) -> Net-(Q1-Pad2)
- Q3 pad 1: Net-(D1-Pad1) -> Net-(D3-Pad1)
- Q3 pad 2: Net-(Q1-Pad2) -> Net-(Q3-Pad2)
Routing:
- net Net-(Q3-Pad2): track 11.9 -> 61.3 mm
- net Net-(Q1-Pad2): track 76.4 -> 28.4 mm
- net Net-(D3-Pad2): track 19.8 -> 18.8 mm
- net Net-(D1-Pad2): track 18.9 -> 19.8 mm
- net Net-(Q2-Pad2): track 48.3 -> 49.1 mm
Changed lines of the file:
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@@
   (general
     (links 75)
-    (no_connects 14)
+    (no_connects 10)
     (area 63.805999 51.613999 152.856001 135.584001)
     (thickness 1.6)
     (drawings 91)
-    (tracks 282)
+    (tracks 280)
     (zones 0)
     (modules 35)
@@
   )
   (module LEDs:LED_1206 (layer F.Cu)
-    (at 69.596 112.649 90)
+    (at 69.596 110.249 90)
     (descr "LED 1206 smd package")
     (tags "LED led 1206 SMD smd SMT smt smdled SMDLED smtled SMTLED")
@@
   )
   (module LEDs:LED_1206 (layer F.Cu)
-    (at 69.596 92.329 90)
+    (at 69.596 94.729 90)
     (descr "LED 1206 smd package")
     (tags "LED led 1206 SMD smd SMT smt smdled SMDLED smtled SMTLED")
@@
   )
   (module TO_SOT_Packages_SMD:SOT-23_Handsoldering (layer F.Cu)
-    (at 76.581 94.869)
+    (at 76.581 97.269)
     (descr "SOT-23, Handsoldering")
     (tags SOT-23)
@@
     (fp_line (start 0.76 1.58) (end -0.7 1.58) (layer F.SilkS) (width 0.12))
     (pad 1 smd rect (at -1.5 -0.95) (size 1.9 0.8) (layers F.Cu F.Paste F.Mask)
-      (net 2 "Net-(D1-Pad1)"))
+      (net 6 "Net-(D3-Pad1)"))
     (pad 2 smd rect (at -1.5 0.95) (size 1.9 0.8) (layers F.Cu F.Paste F.Mask)
-      (net 11 "Net-(Q1-Pad2)"))
+      (net 14 "Net-(Q3-Pad2)"))
     (pad 3 smd rect (at 1.5 0) (size 1.9 0.8) (layers F.Cu F.Paste F.Mask)
       (net 12 GND))
@@
   )
   (module TO_SOT_Packages_SMD:SOT-23_Handsoldering (layer F.Cu)
-    (at 76.581 115.189)
+    (at 76.581 112.789)
     (descr "SOT-23, Handsoldering")
     (tags SOT-23)
@@
     (fp_line (start 0.76 1.58) (end -0.7 1.58) (layer F.SilkS) (width 0.12))
     (pad 1 smd rect (at -1.5 -0.95) (size 1.9 0.8) (layers F.Cu F.Paste F.Mask)
-      (net 6 "Net-(D3-Pad1)"))
+      (net 2 "Net-(D1-Pad1)"))
     (pad 2 smd rect (at -1.5 0.95) (size 1.9 0.8) (layers F.Cu F.Paste F.Mask)
-      (net 14 "Net-(Q3-Pad2)"))
+      (net 11 "Net-(Q1-Pad2)"))
     (pad 3 smd rect (at 1.5 0) (size 1.9 0.8) (layers F.Cu F.Paste F.Mask)
       (net 12 GND))
@@
     (effects (font (size 1.5 1.5) (thickness 0.3)) (justify mirror))
   )
-  (gr_text + (at 70.885 109.7) (layer F.SilkS)
-    (effects (font (size 0.8 0.8) (thickness 0.15)))
-  )
-  (gr_text + (at 70.86 99.525) (layer F.SilkS)
-    (effects (font (size 0.8 0.8) (thickness 0.15)))
-  )
-  (gr_text + (at 70.86 89.375) (layer F.SilkS)
+  (gr_text + (at 67.885 108.55) (layer F.SilkS)
+    (effects (font (size 0.8 0.8) (thickness 0.15)))
+  )
+  (gr_text + (at 67.86 100.775) (layer F.SilkS)
+    (effects (font (size 0.8 0.8) (thickness 0.15)))
+  )
+  (gr_text + (at 67.86 93.025) (layer F.SilkS)
     (effects (font (size 0.8 0.8) (thickness 0.15)))
   )
@@
   (gr_line (start 141.986 135.509) (end 63.881 135.509) (angle 90) (layer Edge.Cuts) (width 0.15))
   (gr_line (start 141.986 135.509) (end 150.876 135.509) (angle 90) (layer Edge.Cuts) (width 0.15))
-  (segment (start 85.471 110.839) (end 88.435 110.839) (width 0.25) (layer F.Cu) (net 1))
-  (segment (start 85.471 110.839) (end 69.756 110.839) (width 0.25) (layer F.Cu) (net 1))
-  (segment (start 69.756 110.839) (end 69.596 110.999) (width 0.25) (layer F.Cu) (net 1))
-  (segment (start 75.081 114.239) (end 69.656 114.239) (width 0.25) (layer F.Cu) (net 2))
-  (segment (start 69.656 114.239) (end 69.596 114.299) (width 0.25) (layer F.Cu) (net 2))
+  (segment (start 69.656 93.919) (end 69.596 93.979) (width 0.25) (layer F.Cu) (net 0))
+  (segment (start 88.435 110.839) (end 80.849 110.839) (width 0.25) (layer F.Cu) (net 1))
+  (segment (start 80.849 110.839) (end 78.609 108.599) (width 0.25) (layer F.Cu) (net 1))
+  (segment (start 78.609 108.599) (end 69.596 108.599) (width 0.25) (layer F.Cu) (net 1))
+  (segment (start 75.081 111.839) (end 69.656 111.839) (width 0.25) (layer F.Cu) (net 2))
   (segment (start 85.471 101.949) (end 88.435 101.949) (width 0.25) (layer F.Cu) (net 3))
   (segment (start 85.471 101.949) (end 83.661 101.949) (width 0.25) (layer F.Cu) (net 3) (status 10))
@@
   (segment (start 75.081 104.079) (end 69.656 104.079) (width 0.25) (layer F.Cu) (net 4) (status 20))
   (segment (start 69.656 104.079) (end 69.596 104.139) (width 0.25) (layer F.Cu) (net 4) (status 30))
+  (segment (start 82.519 93.059) (end 82.499 93.079) (width 0.25) (layer F.Cu) (net 5))
+  (segment (start 82.499 93.079) (end 69.596 93.079) (width 0.25) (layer F.Cu) (net 5))
   (segment (start 88.435 93.059) (end 82.519 93.059) (width 0.25) (layer F.Cu) (net 5))
-  (segment (start 82.519 93.059) (end 80.685 91.225) (width 0.25) (layer F.Cu) (net 5))
-  (segment (start 72.685 91.225) (end 72.139 90.679) (width 0.25) (layer F.Cu) (net 5))
-  (segment (start 80.685 91.225) (end 72.685 91.225) (width 0.25) (layer F.Cu) (net 5))
-  (segment (start 72.139 90.679) (end 69.596 90.679) (width 0.25) (layer F.Cu) (net 5))
-  (segment (start 75.081 93.919) (end 69.656 93.919) (width 0.25) (layer F.Cu) (net 6))
-  (segment (start 69.656 93.919) (end 69.596 93.979) (width 0.25) (layer F.Cu) (net 6))
+  (segment (start 75.081 96.319) (end 69.656 96.319) (width 0.25) (layer F.Cu) (net 6))
   (segment (start 69.385 65.1) (end 69.485 65.2) (width 0.25) (layer B.Cu) (net 7))
   (segment (start 69.485 65.2) (end 69.485 74.774978) (width 0.25) (layer B.Cu) (net 7))
@@
   (segment (start 121.937 132.825) (end 121.435 132.825) (width 0.25) (layer F.Cu) (net 10))
   (via (at 121.435 132.825) (size 0.8) (drill 0.6) (layers F.Cu B.Cu) (net 10))
-  (segment (start 75.081 95.819) (end 70.551 95.819) (width 0.25) (layer F.Cu) (net 11))
-  (segment (start 70.551 95.819) (end 65.935 100.435) (width 0.25) (layer F.Cu) (net 11))
-  (segment (start 73.935 124.225) (end 73.935 125.925) (width 0.25) (layer F.Cu) (net 11))
-  (segment (start 65.935 100.435) (end 65.935 116.225) (width 0.25) (layer F.Cu) (net 11))
-  (segment (start 65.935 116.225) (end 73.935 124.225) (width 0.25) (layer F.Cu) (net 11))
-  (segment (start 73.935 125.925) (end 80.735 132.725) (width 0.25) (layer F.Cu) (net 11))
-  (segment (start 80.735 132.725) (end 87.11341 132.725) (width 0.25) (layer F.Cu) (net 11))
+  (segment (start 75.081 116.139) (end 75.081 113.739) (width 0.25) (layer F.Cu) (net 11))
   (segment (start 87.122 129.54) (end 87.122 131.288) (width 0.25) (layer F.Cu) (net 11))
   (segment (start 87.122 131.288) (end 86.685 131.725) (width 0.25) (layer F.Cu) (net 11))
   (segment (start 86.685 131.725) (end 81.135 131.725) (width 0.25) (layer F.Cu) (net 11))
   (segment (start 81.135 131.725) (end 75.081 125.671) (width 0.25) (layer F.Cu) (net 11))
-  (segment (start 87.11341 132.725) (end 88.61341 131.225) (width 0.25) (layer F.Cu) (net 11))
-  (segment (start 88.61341 131.225) (end 90.517 131.225) (width 0.25) (layer F.Cu) (net 11))
+  (segment (start 75.081 125.671) (end 75.081 116.139) (width 0.25) (layer F.Cu) (net 11))
   (segment (start 138.249 93.529) (end 138.249 98.114) (width 0.4) (layer F.Cu) (net 12))
   (segment (start 143.635 95.463) (end 141.141 95.463) (width 0.4) (layer F.Cu) (net 12))
@@
   (segment (start 120.142 129.54) (end 120.269 129.54) (width 0.25) (layer F.Cu) (net 12))
   (segment (start 149.635 95.463) (end 149.635 93.725) (width 0.4) (layer F.Cu) (net 12))
-  (segment (start 75.081 105.979) (end 70.551 105.979) (width 0.25) (layer F.Cu) (net 13))
-  (segment (start 70.551 105.979) (end 66.421 110.109) (width 0.25) (layer F.Cu) (net 13))
-  (segment (start 66.421 110.109) (end 66.421 116.07459) (width 0.25) (layer F.Cu) (net 13))
+  (segment (start 75.081 105.979) (end 69.181 105.979) (width 0.25) (layer F.Cu) (net 13))
+  (segment (start 74.435 125.725) (end 80.935 132.225) (width 0.25) (layer F.Cu) (net 13))
+  (segment (start 69.181 105.979) (end 66.421 108.739) (width 0.25) (layer F.Cu) (net 13))
+  (segment (start 66.421 108.739) (end 66.421 116.07459) (width 0.25) (layer F.Cu) (net 13))
   (segment (start 66.421 116.07459) (end 74.435 124.08859) (width 0.25) (layer F.Cu) (net 13))
   (segment (start 74.435 124.08859) (end 74.435 125.725) (width 0.25) (layer F.Cu) (net 13))
-  (segment (start 74.435 125.725) (end 80.935 132.225) (width 0.25) (layer F.Cu) (net 13))
   (segment (start 80.935 132.225) (end 86.977 132.225) (width 0.25) (layer F.Cu) (net 13))
+  (segment (start 86.977 132.225) (end 88.812001 130.389999) (width 0.25) (layer F.Cu) (net 13))
   (segment (start 88.812001 130.389999) (end 89.662 129.54) (width 0.25) (layer F.Cu) (net 13))
-  (segment (start 86.977 132.225) (end 88.812001 130.389999) (width 0.25) (layer F.Cu) (net 13))
+  (segment (start 65.935 100.435) (end 68.151 98.219) (width 0.25) (layer F.Cu) (net 14))
+  (segment (start 68.151 98.219) (end 75.081 98.219) (width 0.25) (layer F.Cu) (net 14))
+  (segment (start 73.935 124.225) (end 73.935 125.925) (width 0.25) (layer F.Cu) (net 14))
+  (segment (start 65.935 100.435) (end 65.935 116.225) (width 0.25) (layer F.Cu) (net 14))
+  (segment (start 65.935 116.225) (end 73.935 124.225) (width 0.25) (layer F.Cu) (net 14))
+  (segment (start 73.935 125.925) (end 80.735 132.725) (width 0.25) (layer F.Cu) (net 14))
+  (segment (start 80.735 132.725) (end 87.11341 132.725) (width 0.25) (layer F.Cu) (net 14))
+  (segment (start 87.11341 132.725) (end 88.61341 131.225) (width 0.25) (layer F.Cu) (net 14))
+  (segment (start 88.61341 131.225) (end 90.517 131.225) (width 0.25) (layer F.Cu) (net 14))
   (segment (start 90.517 131.225) (end 92.202 129.54) (width 0.25) (layer F.Cu) (net 14))
-  (segment (start 75.081 125.671) (end 75.081 116.139) (width 0.25) (layer F.Cu) (net 14))
   (segment (start 125.2171 118.1276) (end 125.2171 121.1531) (width 0.25) (layer F.Cu) (net 21) (status 10))
   (segment (start 114.808 124.714) (end 112.522 127) (width 0.25) (layer F.Cu) (net 21))
