File: backplane.kicad_pcb (KiCad board)
At the start: 2 copper layers, 88.9 x 83.8 mm, 35 parts, among them J1 I2C, J2 I2C, J3 SER, J4 PWR, J5 PWR, J6 FAN, Q1 Q_NMOS_DGS, Q2 Q_NMOS_DGS, Q3 Q_NMOS_DGS, Q4 Q_NMOS_DGS, U1 Raspberry_Pi_2_3, U2 IC880A-SPI, U3 SHT21, U4 MP1584_MODULE

Commit message: Improvements
Parts:
- moved G*** 14.2 mm to (111.4, 95.2)
- moved J3 0.54 mm to (75.1, 131.9)
Routing:
- net /3.3V: track 287.7 -> 248.4 mm
Other:
- board text added: "(Optional)"

Commit message: Improvements
Routing:
- net Net-(Q4-Pad2): track 114.0 -> 107.8 mm
Changed lines of the file:
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@@
   (general
     (links 75)
-    (no_connects 10)
+    (no_connects 9)
     (area 63.805999 51.613999 152.856001 135.584001)
     (thickness 1.6)
     (drawings 92)
-    (tracks 279)
+    (tracks 278)
     (zones 0)
     (modules 35)
@@
   (layers
     (0 F.Cu signal)
-    (31 B.Cu signal hide)
+    (31 B.Cu signal)
     (32 B.Adhes user)
     (33 F.Adhes user)
@@
   (segment (start 80.435 61.275) (end 80.435 57.225) (width 0.25) (layer F.Cu) (net 52))
   (segment (start 80.435 57.225) (end 79.435 56.225) (width 0.25) (layer F.Cu) (net 52))
+  (segment (start 92.685 123.225) (end 86.685 123.225) (width 0.25) (layer B.Cu) (net 53))
+  (segment (start 86.685 123.225) (end 84.185 120.725) (width 0.25) (layer B.Cu) (net 53))
+  (segment (start 84.185 120.725) (end 84.185 113.475) (width 0.25) (layer B.Cu) (net 53))
+  (segment (start 84.185 113.475) (end 85.935 111.725) (width 0.25) (layer B.Cu) (net 53))
+  (segment (start 85.935 111.725) (end 85.935 77.399264) (width 0.25) (layer B.Cu) (net 53))
+  (segment (start 85.935 77.399264) (end 85.935 76.975) (width 0.25) (layer B.Cu) (net 53))
+  (segment (start 84.734999 70.524999) (end 84.435 70.225) (width 0.25) (layer F.Cu) (net 53))
+  (segment (start 85.935 76.824998) (end 85.935 71.725) (width 0.25) (layer F.Cu) (net 53))
+  (segment (start 80.435 66.225) (end 84.435 70.225) (width 0.25) (layer B.Cu) (net 53))
+  (segment (start 85.935 71.725) (end 84.734999 70.524999) (width 0.25) (layer F.Cu) (net 53))
+  (via (at 84.435 70.225) (size 0.6) (drill 0.4) (layers F.Cu B.Cu) (net 53))
+  (segment (start 85.885001 77.024999) (end 85.935 76.975) (width 0.25) (layer F.Cu) (net 53))
+  (via (at 85.935 76.975) (size 0.6) (drill 0.4) (layers F.Cu B.Cu) (net 53))
   (segment (start 122.682 129.54) (end 123.935 128.287) (width 0.25) (layer F.Cu) (net 53))
   (segment (start 123.935 128.287) (end 123.935 123.725) (width 0.25) (layer F.Cu) (net 53))
-  (segment (start 92.685 123.225) (end 87.185 123.225) (width 0.25) (layer B.Cu) (net 53))
-  (segment (start 87.185 123.225) (end 84.185 120.225) (width 0.25) (layer B.Cu) (net 53))
-  (segment (start 84.185 120.225) (end 84.185 117.475) (width 0.25) (layer B.Cu) (net 53))
-  (segment (start 90.435 78.725) (end 88.435 76.725) (width 0.25) (layer B.Cu) (net 53))
-  (segment (start 84.185 117.475) (end 88.234991 113.425009) (width 0.25) (layer B.Cu) (net 53))
-  (segment (start 88.234991 113.425009) (end 89.871401 113.425009) (width 0.25) (layer B.Cu) (net 53))
-  (segment (start 89.871401 113.425009) (end 90.435 112.86141) (width 0.25) (layer B.Cu) (net 53))
-  (segment (start 90.435 112.86141) (end 90.435 78.725) (width 0.25) (layer B.Cu) (net 53))
   (segment (start 95.435 123.225) (end 92.685 123.225) (width 0.25) (layer F.Cu) (net 53))
   (via (at 92.685 123.225) (size 0.6) (drill 0.4) (layers F.Cu B.Cu) (net 53))
@@
   (via (at 123.935 123.725) (size 0.6) (drill 0.4) (layers F.Cu B.Cu) (net 53))
   (segment (start 80.435 66.225) (end 80.435 63.175) (width 0.25) (layer F.Cu) (net 53))
-  (segment (start 88.435 71.225) (end 83.435 66.225) (width 0.25) (layer B.Cu) (net 53))
-  (segment (start 83.435 66.225) (end 80.435 66.225) (width 0.25) (layer B.Cu) (net 53))
   (via (at 80.435 66.225) (size 0.6) (drill 0.4) (layers F.Cu B.Cu) (net 53))
-  (segment (start 88.435 73.725) (end 88.435 71.225) (width 0.25) (layer B.Cu) (net 53))
-  (via (at 88.435 73.725) (size 0.6) (drill 0.4) (layers F.Cu B.Cu) (net 53))
-  (segment (start 88.435 76.725) (end 88.435 73.725) (width 0.25) (layer F.Cu) (net 53))
-  (via (at 88.435 76.725) (size 0.6) (drill 0.4) (layers F.Cu B.Cu) (net 53))
   (zone (net 12) (net_name GND) (layer B.Cu) (hatch edge 0.508)
     (connect_pads (clearance 0.508))

Commit message: Integrate step-down module
Parts:
- turned U4 to 0 degrees
Connections:
- U4 pad 1: /5V -> Net-(J5-Pad1)
- U4 pad 2: GND -> Net-(J5-Pad2)
- U4 pad 3: Net-(J5-Pad1) -> /5V
- U4 pad 4: Net-(J5-Pad2) -> GND
Routing:
- net Net-(J5-Pad2): track 0.00 -> 129.8 mm, vias 0 -> 3
- net Net-(J5-Pad1): track 0.00 -> 102.4 mm, vias 0 -> 3
- net /5V: track 267.5 -> 301.5 mm
- net Net-(J3-Pad1): track 48.9 -> 65.6 mm, vias 1 -> 0
- net Net-(J3-Pad2): track 45.7 -> 55.7 mm, vias 1 -> 0
- net GND: track 24.4 -> 26.9 mm
- net Net-(Q4-Pad2): track 107.8 -> 106.4 mm

Commit message: Improvements
Routing:
- net /5V: track 301.5 -> 299.9 mm
Changed lines of the file:
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@@
     (thickness 1.6)
     (drawings 92)
-    (tracks 318)
+    (tracks 321)
     (zones 0)
     (modules 35)
@@
   (segment (start 117.602 123.698) (end 110.744 123.698) (width 0.25) (layer F.Cu) (net 24))
   (segment (start 120.1371 121.1629) (end 117.602 123.698) (width 0.25) (layer F.Cu) (net 24))
+  (segment (start 81.885001 116.774999) (end 82.185 116.475) (width 0.25) (layer B.Cu) (net 25))
+  (segment (start 77.685 120.975) (end 81.885001 116.774999) (width 0.25) (layer B.Cu) (net 25))
+  (segment (start 105.507 131.475) (end 80.88752 131.475) (width 0.25) (layer B.Cu) (net 25))
+  (segment (start 77.685 128.27248) (end 77.685 120.975) (width 0.25) (layer B.Cu) (net 25))
+  (segment (start 80.88752 131.475) (end 77.685 128.27248) (width 0.25) (layer B.Cu) (net 25))
   (segment (start 107.442 129.54) (end 105.507 131.475) (width 0.25) (layer B.Cu) (net 25))
-  (segment (start 77.685 120.975) (end 82.185 116.475) (width 0.25) (layer B.Cu) (net 25))
-  (segment (start 105.507 131.475) (end 80.885 131.475) (width 0.25) (layer B.Cu) (net 25))
-  (segment (start 80.885 131.475) (end 77.685 128.275) (width 0.25) (layer B.Cu) (net 25))
-  (segment (start 77.685 128.275) (end 77.685 120.975) (width 0.25) (layer B.Cu) (net 25))
   (segment (start 82.185 116.475) (end 83.725 114.935) (width 0.25) (layer F.Cu) (net 25))
   (segment (start 83.725 114.935) (end 124.5645 114.935) (width 0.25) (layer F.Cu) (net 25))
@@
   (segment (start 133.135 86.325) (end 133.135 85.425) (width 0.4) (layer F.Cu) (net 44))
   (segment (start 133.135 85.425) (end 131.985 84.275) (width 0.4) (layer F.Cu) (net 44))
-  (segment (start 131.699 132.334) (end 129.6035 134.4295) (width 0.8) (layer B.Cu) (net 45))
-  (segment (start 129.6035 134.4295) (end 81.3395 134.4295) (width 0.8) (layer B.Cu) (net 45))
-  (segment (start 81.3395 134.4295) (end 64.77 117.86) (width 0.8) (layer B.Cu) (net 45))
-  (segment (start 64.77 117.86) (end 64.77 89.8) (width 0.8) (layer B.Cu) (net 45))
+  (segment (start 131.122336 132.3594) (end 131.8514 132.3594) (width 0.8) (layer F.Cu) (net 45))
+  (segment (start 132.842 131.3688) (end 132.842 129.54) (width 0.8) (layer F.Cu) (net 45))
+  (segment (start 131.8514 132.3594) (end 132.842 131.3688) (width 0.8) (layer F.Cu) (net 45))
+  (via (at 131.122336 132.3594) (size 1) (drill 0.8) (layers F.Cu B.Cu) (net 45))
+  (segment (start 64.77 89.8) (end 64.77 117.86) (width 0.8) (layer B.Cu) (net 45))
+  (segment (start 64.77 117.86) (end 67.1282 120.2182) (width 0.8) (layer B.Cu) (net 45))
+  (segment (start 67.1282 120.2182) (end 68.4022 120.2182) (width 0.8) (layer B.Cu) (net 45))
+  (segment (start 68.4022 120.2182) (end 80.5434 132.3594) (width 0.8) (layer B.Cu) (net 45))
+  (segment (start 80.5434 132.3594) (end 131.122336 132.3594) (width 0.8) (layer B.Cu) (net 45))
   (segment (start 66.421 87.979) (end 64.77 89.63) (width 0.8) (layer B.Cu) (net 45))
   (segment (start 64.77 89.63) (end 64.77 74.09) (width 0.8) (layer B.Cu) (net 45))
@@
   (segment (start 89.6171 56.8276) (end 89.535 56.9097) (width 0.8) (layer F.Cu) (net 45))
   (segment (start 89.535 56.9097) (end 89.535 64.135) (width 0.8) (layer F.Cu) (net 45))
-  (segment (start 132.842 129.54) (end 132.842 131.064) (width 0.8) (layer F.Cu) (net 45))
-  (segment (start 132.842 131.064) (end 131.699 132.334) (width 0.8) (layer F.Cu) (net 45))
-  (via (at 131.699 132.334) (size 0.6) (drill 0.4) (layers F.Cu B.Cu) (net 45))
   (segment (start 132.842 129.54) (end 135.382 129.54) (width 0.8) (layer F.Cu) (net 45))
   (segment (start 135.636 129.794) (end 135.382 129.54) (width 0.25) (layer F.Cu) (net 45))

Commit message: Start working on variant
Parts:
- added C2: C, capacitor-unmarked:CAP_UNMARKED, F.Cu at (102.9, 62.2)
- moved G*** 114.5 mm to (225.0, 81.2)
- moved J1 92.3 mm to (153.7, 108.0)
- moved J2 87.7 mm to (153.7, 71.1)
- moved J4 82.5 mm to (67.1, 123.6), turned to 270 degrees
- moved J6 74.4 mm to (153.7, 61.6), turned to 0 degrees
- moved D4 69.9 mm to (146.4, 67.9), turned to 180 degrees
- moved J5 62.1 mm to (67.1, 61.5)
- moved Q4 61.3 mm to (143.3, 62.5)
- moved U4 40.5 mm to (85.2, 67.2)
Routing:
- net /5V: track 299.9 -> 163.3 mm, vias 2 -> 0
- net Net-(J5-Pad2): track 129.8 -> 14.4 mm, vias 3 -> 0
- net Net-(J1-Pad1): track 148.3 -> 41.1 mm
- net Net-(Q4-Pad2): track 106.4 -> 0.00 mm, vias 6 -> 0
- net Net-(J1-Pad2): track 150.8 -> 51.8 mm, vias 3 -> 2
- net Net-(J5-Pad1): track 102.4 -> 11.7 mm, vias 3 -> 0
- net /3.3V: track 248.4 -> 206.0 mm
- net Net-(D4-Pad2): track 9.74 -> 19.8 mm
Other:
- board size 88.9 x 83.8 mm -> 93.9 x 83.8 mm
- board text added: "Capacitor (Optional)"
- board text added: "MP1584 Module (Optional)"
- board text removed: "(Optional)"
- board text removed: "PWR (Conv)"

Commit message: More routing
Parts:
- added R6: R, Resistors_SMD:R_1206_HandSoldering, F.Cu at (79.9, 119.0)
- added R7: R, Resistors_SMD:R_1206_HandSoldering, F.Cu at (96.3, 108.7)
- added R8: R, Resistors_SMD:R_1206_HandSoldering, F.Cu at (40.0, 116.5)
- C2: footprint capacitor-unmarked:CAP_UNMARKED -> Capacitors_THT:CP_Radial_D12.5mm_P7.50mm
- R4, R5: footprint Capacitors_SMD:C_1206 -> Resistors_SMD:R_1206_HandSoldering
- moved R5 1.56 mm to (131.6, 87.9)
- moved C1 0.84 mm to (148.8, 91.7)
- moved U3 0.73 mm to (143.6, 92.5)
Routing:
- net Net-(Q4-Pad2): track 0.00 -> 83.5 mm, vias 0 -> 2
- net Net-(J1-Pad1): track 41.1 -> 81.6 mm
- net /3.3V: track 206.0 -> 244.0 mm
- net /5V: track 163.3 -> 193.2 mm
- net Net-(J1-Pad2): track 51.8 -> 67.3 mm
- net Net-(Q1-Pad2): track 28.4 -> 31.2 mm
- net GND: track 26.9 -> 25.0 mm
Other:
- outline, holes or cut-outs redrawn

Commit message: Finish routing
Parts:
- moved J3 130.9 mm to (205.2, 146.4), turned to 180 degrees
- moved R8 101.5 mm to (141.5, 117.7)
- moved R1 64.4 mm to (150.2, 127.3)
- moved R2 64.4 mm to (150.2, 118.4)
- moved R3 64.4 mm to (150.2, 109.5)
- moved G*** 57.4 mm to (171.6, 102.0)
- moved J1 54.8 mm to (205.2, 126.4)
- moved J2 54.8 mm to (205.2, 89.5)
- moved J6 54.8 mm to (205.2, 80.0)
- moved Q4 54.8 mm to (194.8, 81.0)
- moved REF** 54.8 mm to (200.7, 150.4)
- moved REF** 54.8 mm to (200.7, 74.0)
- moved U3 54.8 mm to (195.2, 110.9)
- moved D1 54.8 mm to (121.2, 128.7)
- moved D2 54.8 mm to (121.2, 120.9)
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Routing:
- net /5V: track 193.2 -> 280.9 mm, vias 0 -> 1
- net Net-(J1-Pad2): track 67.3 -> 106.4 mm
- net Net-(J1-Pad1): track 81.6 -> 120.1 mm
- net Net-(J3-Pad1): track 65.6 -> 27.9 mm
- net Net-(J3-Pad2): track 55.7 -> 37.8 mm
- net Net-(Q2-Pad2): track 49.1 -> 63.0 mm
- net Net-(Q3-Pad2): track 61.2 -> 74.6 mm
- net /3.3V: track 244.0 -> 233.8 mm
- net Net-(D3-Pad2): track 18.8 -> 29.0 mm
- net Net-(D2-Pad2): track 19.3 -> 29.5 mm
- net Net-(D1-Pad2): track 19.8 -> 29.9 mm
- net GND: track 25.0 -> 31.2 mm
- net Net-(U1-Pad24): track 93.1 -> 90.1 mm
Other:
- outline, holes or cut-outs redrawn
