File: backplane.sch (KiCad schematic (older format))
At the start: 35 parts, among them J1 I2C, J2 I2C, J3 SER, J4 PWR, J5 PWR, J6 FAN, J7 Conn_PPS, Q4 Q_NMOS_GSD, Q5 Q_PMOS_GSD, SW1 SW_Push, U1 Raspberry_Pi_2_3, U2 IC880A-SPI, U3 SHT21, U4 MP1584_MODULE, U5 MCP3425A0T-E/CH

Commit message: More Swissness :wink:
Parts:
- J7: value Conn_PPS -> PPS
Changed lines of the file:
@@
 P 4150 7500
 F 0 "J7" H 4150 7600 50  0000 C CNN
-F 1 "Conn_PPS" H 4150 7400 50  0000 C CNN
+F 1 "PPS" H 4150 7400 50  0000 C CNN
 F 2 "headers:header_1x1_unmarked" H 4150 7500 50  0001 C CNN
 F 3 "" H 4150 7500 50  0001 C CNN

Commit message: Increase 2x20 pin header restrings (#23)
Also update LED resistor values
Parts:
- R1: value 27Ω 1/8W -> 82Ω 1/8W
- R2: value 270Ω 1/8W -> 330Ω 1/8W
- R3: value 330Ω 1/8W -> 220Ω 1/8W
- U1: footprint Pin_Headers:Pin_Header_Straight_2x20_Pitch2.54mm -> headers:Pin_Header_Straight_2x20_Pitch2.54mm
Changed lines of the file:
@@
 F 0 "U1" H 2800 4550 50  0000 C CNN
 F 1 "Raspberry_Pi_2_3" H 1700 6700 50  0000 C CNN
-F 2 "Pin_Headers:Pin_Header_Straight_2x20_Pitch2.54mm" H 3100 7050 50  0001 C CNN
+F 2 "headers:Pin_Header_Straight_2x20_Pitch2.54mm" H 3100 7050 50  0001 C CNN
 F 3 "" H 2150 5650 50  0001 C CNN
 	1    2100 5800
@@
 P 1700 2400
 F 0 "R3" V 1780 2400 50  0000 C CNN
-F 1 "330Ω 1/8W" V 1600 2400 50  0000 C CNN
+F 1 "220Ω 1/8W" V 1600 2400 50  0000 C CNN
 F 2 "Resistors_SMD:R_1206" V 1630 2400 50  0001 C CNN
 F 3 "" H 1700 2400 50  0000 C CNN
@@
 P 1700 2000
 F 0 "R2" V 1780 2000 50  0000 C CNN
-F 1 "270Ω 1/8W" V 1600 2000 50  0000 C CNN
+F 1 "330Ω 1/8W" V 1600 2000 50  0000 C CNN
 F 2 "Resistors_SMD:R_1206" V 1630 2000 50  0001 C CNN
 F 3 "" H 1700 2000 50  0000 C CNN
@@
 P 1700 1600
 F 0 "R1" V 1780 1600 50  0000 C CNN
-F 1 "27Ω 1/8W" V 1600 1600 50  0000 C CNN
+F 1 "82Ω 1/8W" V 1600 1600 50  0000 C CNN
 F 2 "Resistors_SMD:R_1206" V 1630 1600 50  0001 C CNN
 F 3 "" H 1700 1600 50  0000 C CNN

Commit message: Update for Zvepower regulator
It has castellated edges and is slightly smaller.
Parts:
- U4: footprint regulators:MP1584_MODULE -> regulators:MP1584_MODULE_ZVEPOWER
Connections:
- net GND: now also U4.4 (OUT-)
- net at C2.2, D6.2 (A), F1.1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: now also U4.3 (OUT+)
- net at U4.1 (IN-): now also J5.1 (GND)
- net at U4.2 (IN+): now also D6.1 (K), J5.2 (VCC), U4.5 (EN)
Other:
- moved on the sheet: D6, U4
Changed lines of the file:
@@
 Sheet 1 1
 Title "iC880A RPi Backplane"
-Date "2018-01-17"
-Rev "v1.5"
+Date "2018-03-26"
+Rev "v1.6"
 Comp "Danilo Bargen / Coredump Rapperswil"
 Comment1 "Buy from https://shop.coredump.ch/"
@@
 L MP1584_MODULE U4
 U 1 1 589F7FAA
-P 8700 1200
-F 0 "U4" H 8700 950 60  0000 C CNN
-F 1 "MP1584_MODULE" H 8700 1500 60  0000 C CNN
-F 2 "regulators:MP1584_MODULE" H 8700 1200 60  0001 C CNN
-F 3 "" H 8700 1200 60  0001 C CNN
-	1    8700 1200
+P 8700 1100
+F 0 "U4" H 9050 800 60  0000 C CNN
+F 1 "MP1584_MODULE" H 8700 1450 60  0000 C CNN
+F 2 "regulators:MP1584_MODULE_ZVEPOWER" H 8700 1100 60  0001 C CNN
+F 3 "" H 8700 1100 60  0001 C CNN
+	1    8700 1100
 	1    0    0    1
 $EndComp
@@
 L D D6
 U 1 1 58F9565C
-P 8700 750
-F 0 "D6" H 8550 700 50  0000 C CNN
-F 1 "D" H 8800 700 50  0000 C CNN
-F 2 "DO214:DO-214AC" H 8700 750 50  0001 C CNN
-F 3 "http://mikroshop.ch/pdf/ss12.pdf" H 8700 750 50  0001 C CNN
-F 4 "Vishay SS14" H 8700 750 60  0001 C CNN "Model"
-	1    8700 750
+P 8700 700
+F 0 "D6" H 8550 650 50  0000 C CNN
+F 1 "D" H 8800 650 50  0000 C CNN
+F 2 "DO214:DO-214AC" H 8700 700 50  0001 C CNN
+F 3 "http://mikroshop.ch/pdf/ss12.pdf" H 8700 700 50  0001 C CNN
+F 4 "Vishay SS14" H 8700 700 60  0001 C CNN "Model"
+	1    8700 700
 	1    0    0    -1
 $EndComp
@@
 	8100 1100 8250 1100
 Wire Wire Line
-	8100 1200 8100 1300
-Wire Wire Line
-	8100 1300 8250 1300
-Wire Wire Line
-	8200 750  8550 750
-Wire Wire Line
-	8850 750  9200 750
+	8200 700  8550 700
+Wire Wire Line
+	8850 700  9200 700
 Wire Wire Line
 	9150 1100 9700 1100
 Wire Wire Line
-	9150 1300 9250 1300
-Wire Wire Line
-	9250 1300 9250 1500
+	9150 1250 9250 1250
+Wire Wire Line
+	9250 1250 9250 1500
 Wire Wire Line
 	9450 1100 9450 1150
@@
 Connection ~ 9450 1800
 Wire Wire Line
-	8200 750  8200 1100
+	8200 700  8200 1100
 Connection ~ 8200 1100
 Wire Wire Line
-	9200 750  9200 1100
+	9200 700  9200 1100
 Connection ~ 9200 1100
 Wire Wire Line
@@
 	1    0    0    -1
 $EndComp
+Wire Wire Line
+	8250 950  8200 950
+Connection ~ 8200 950
+Wire Wire Line
+	8100 1200 8200 1200
+Wire Wire Line
+	8200 1200 8200 1250
+Wire Wire Line
+	8200 1250 8250 1250
 $EndSCHEMATC

Commit message: Schematics: Add SHTC1
Parts:
- removed U3: SHT21, sensirion:SHT21, symbol SHT21
- added U3: SHTC1, sensirion:SHTC1, symbol SHTC1
Connections:
- net 3.3V: now also U3.1 (VDD)
- net GND: now also U3.4 (VSS)
- net SCL: now also U3.2 (SCL)
- net SDA: now also U3.3 (SDA)
Other:
- note added: "SHTC1 Sensor"
- note added: "The Sensirion SHTC1 sensor\nmeasures both temperature\nand humidity.\n\nTemperature\nmeasurements\nare accurate to\n±0.3°C, humidity is\naccurate to ±3%RH."
- note removed: "SHT21 Sensor"
- note removed: "The Sensirion SHT21 sensor\nmeasures both temperature\nand humidity.\n\nTemperature\nmeasurements\nare accurate to\n±0.3°C, humidity is\naccurate to ±2%RH."
- moved on the sheet: R4, R5
Changed lines of the file:
@@
 EESchema Schematic File Version 2
 LIBS:backplane-rescue
-LIBS:power
-LIBS:device
-LIBS:transistors
-LIBS:conn
-LIBS:linear
-LIBS:regul
-LIBS:74xx
-LIBS:cmos4000
-LIBS:adc-dac
-LIBS:memory
-LIBS:xilinx
-LIBS:microcontrollers
-LIBS:dsp
-LIBS:microchip
-LIBS:analog_switches
-LIBS:motorola
-LIBS:texas
-LIBS:intel
-LIBS:audio
-LIBS:interface
-LIBS:digital-audio
-LIBS:philips
-LIBS:display
-LIBS:cypress
-LIBS:siliconi
-LIBS:opto
-LIBS:atmel
-LIBS:contrib
-LIBS:valves
 LIBS:ic880a-spi
 LIBS:headers
@@
 LIBS:sensirion
 LIBS:regulators
-LIBS:switches
 LIBS:backplane-cache
 EELAYER 25 0
@@
 Sheet 1 1
 Title "iC880A RPi Backplane"
-Date "2018-03-26"
-Rev "v1.6"
+Date "2018-04-23"
+Rev "v2.0"
 Comp "Danilo Bargen / Coredump Rapperswil"
 Comment1 "Buy from https://shop.coredump.ch/"
@@
 NoConn ~ 6900 4650
 $Comp
-L SHT21 U3
-U 1 1 5898B996
-P 6150 1500
-F 0 "U3" H 6150 1200 60  0000 C CNN
-F 1 "SHT21" H 6150 1800 60  0000 C CNN
-F 2 "sensirion:SHT21" H 6150 1500 60  0001 C CNN
-F 3 "https://www.sensirion.com/fileadmin/user_upload/customers/sensirion/Dokumente/2_Humidity_Sensors/Sensirion_Humidity_Sensors_SHT21_Datasheet_V4.pdf" H 6150 1500 60  0001 C CNN
-	1    6150 1500
-	1    0    0    -1
-$EndComp
-$Comp
 L C C1
 U 1 1 5898C4BA
@@
 L R R4
 U 1 1 589B82C4
-P 6650 1900
-F 0 "R4" V 6730 1900 40  0000 C CNN
-F 1 "R" V 6657 1901 40  0000 C CNN
-F 2 "Resistors_SMD:R_1206" V 6580 1900 30  0001 C CNN
-F 3 "" H 6650 1900 30  0000 C CNN
-F 4 "10kΩ" V 6550 1900 60  0000 C CNN "R"
-	1    6650 1900
+P 6650 1950
+F 0 "R4" V 6730 1950 40  0000 C CNN
+F 1 "R" V 6657 1951 40  0000 C CNN
+F 2 "Resistors_SMD:R_1206" V 6580 1950 30  0001 C CNN
+F 3 "" H 6650 1950 30  0000 C CNN
+F 4 "10kΩ" V 6550 1950 60  0000 C CNN "R"
+	1    6650 1950
 	-1   0    0    1
 $EndComp
@@
 L R R5
 U 1 1 589B831C
-P 5650 1900
-F 0 "R5" V 5730 1900 40  0000 C CNN
-F 1 "R" V 5657 1901 40  0000 C CNN
-F 2 "Resistors_SMD:R_1206" V 5580 1900 30  0001 C CNN
-F 3 "" H 5650 1900 30  0000 C CNN
-F 4 "10kΩ" V 5550 1900 60  0000 C CNN "R"
-	1    5650 1900
+P 5650 1950
+F 0 "R5" V 5730 1950 40  0000 C CNN
+F 1 "R" V 5657 1951 40  0000 C CNN
+F 2 "Resistors_SMD:R_1206" V 5580 1950 30  0001 C CNN
+F 3 "" H 5650 1950 30  0000 C CNN
+F 4 "10kΩ" V 5550 1950 60  0000 C CNN "R"
+	1    5650 1950
 	-1   0    0    1
 $EndComp
@@
 Text GLabel 2300 4350 2    60   Input ~ 0
 3.3V
-Text GLabel 6700 1650 2    60   Input ~ 0
+Text GLabel 6700 1700 2    60   Input ~ 0
 SDA
-Text GLabel 6650 2100 3    60   Input ~ 0
+Text GLabel 6650 2150 3    60   Input ~ 0
 3.3V
 $Comp
@@
 	1    0    0    -1
 $EndComp
-Text GLabel 5650 2100 3    60   Input ~ 0
+Text GLabel 5650 2150 3    60   Input ~ 0
 3.3V
-Text GLabel 5600 1650 0    60   Input ~ 0
+Text GLabel 5600 1700 0    60   Input ~ 0
 SCL
 Text GLabel 3100 4900 2    60   Input ~ 0
@@
 LEDs
 Text Notes 3750 800  0    157  ~ 0
-SHT21 Sensor
+SHTC1 Sensor
 Text Notes 4150 2850 0    157  ~ 0
 I²C Breakouts
@@
 The board includes a 5V\npower input/output\nconnector as well as a\nMP1584 step-down\nvoltage regulator for\n6.7-28V input.
 Text Notes 3750 1800 0    60   ~ 0
-The Sensirion SHT21 sensor\nmeasures both temperature\nand humidity.\n\nTemperature\nmeasurements\nare accurate to\n±0.3°C, humidity is\naccurate to ±2%RH.
+The Sensirion SHTC1 sensor\nmeasures both temperature\nand humidity.\n\nTemperature\nmeasurements\nare accurate to\n±0.3°C, humidity is\naccurate to ±3%RH.
 Text Notes 7500 5000 0    157  ~ 0
 Button
@@
 	3100 6500 3000 6500
 Wire Wire Line
-	5400 1500 5650 1500
+	5400 1500 5700 1500
 Connection ~ 2200 4450
 Wire Wire Line
@@
 	3000 5000 3050 5000
 Wire Wire Line
-	5650 1650 5600 1650
-Wire Wire Line
-	5650 2100 5650 2050
-Wire Wire Line
-	5650 1650 5650 1750
+	5600 1700 5700 1700
+Wire Wire Line
+	5650 2150 5650 2100
+Wire Wire Line
+	5650 1700 5650 1800
 Wire Wire Line
 	7050 1500 7050 1550
 Wire Wire Line
-	6650 1500 7050 1500
-Wire Wire Line
-	6650 2100 6650 2050
-Wire Wire Line
-	6650 1650 6650 1750
-Wire Wire Line
-	6700 1650 6650 1650
+	6600 1500 7050 1500
+Wire Wire Line
+	6650 2150 6650 2100
+Wire Wire Line
+	6650 1700 6650 1800
+Wire Wire Line
+	6600 1700 6700 1700
 Wire Wire Line
 	1650 7400 1650 7500
@@
 Wire Wire Line
 	8200 1250 8250 1250
+$Comp
+L SHTC1 U3
+U 1 1 5ADE2706
+P 6150 1600
+F 0 "U3" H 6150 1300 60  0000 C CNN
+F 1 "SHTC1" H 6150 1900 60  0000 C CNN
+F 2 "sensirion:SHTC1" H 6150 1600 60  0001 C CNN
+F 3 "" H 6150 1600 60  0001 C CNN
+	1    6150 1600
+	1    0    0    -1
+$EndComp
+Connection ~ 5650 1700
+Connection ~ 6650 1700
 $EndSCHEMATC

Commit message: Add SHTC3 in parallel to SHT21
Parts:
- removed U3: SHTC1, sensirion:SHTC1, symbol SHTC1
- added U3: SHT21, sensirion:SHT21, symbol SHT21
- added U6: SHTC3, sensirion:SHTC1, symbol SHTC3
Connections:
- net 3.3V: now also U3.5 (VDD), U6.1 (VDD)
- net GND: now also U3.2 (VSS), U6.4 (VSS)
- net SCL: now also U3.6 (SCL), U6.2 (SCL)
- net SDA: now also U3.1 (SDA), U6.3 (SDA)
Other:
- note added: "Accuracy SHT21:\n±0.3°C / ±3%RH"
- note added: "Accuracy SHTC3:\n±0.2°C / ±2%RH"
- note added: "I²C Pull-Ups"
- note added: "SHTC1 Sensors"
- note added: "The Sensirion SHT21/SHTC3 sensor\nmeasures both temperature\nand humidity."
- note removed: "SHTC1 Sensor"
- note removed: "The Sensirion SHTC1 sensor\nmeasures both temperature\nand humidity.\n\nTemperature\nmeasurements\nare accurate to\n±0.3°C, humidity is\naccurate to ±3%RH."
- moved on the sheet: C1, R4, R5

Commit message: Update schematics
Other:
- note added: "SHTC3 Sensor"
- note added: "The Sensirion SHT21/SHTC3 sensors\nmeasure both temperature\nand humidity."
- note removed: "SHTC1 Sensors"
- note removed: "The Sensirion SHT21/SHTC3 sensor\nmeasures both temperature\nand humidity."
Changed lines of the file:
@@
 LEDs
 Text Notes 3200 750  0    157  ~ 0
-SHTC1 Sensors
+SHTC3 Sensor
 Text Notes 4150 2850 0    157  ~ 0
 I²C Breakouts
@@
 The board includes a 5V\npower input/output\nconnector as well as a\nMP1584 step-down\nvoltage regulator for\n6.7-28V input.
 Text Notes 3200 1100 0    60   ~ 0
-The Sensirion SHT21/SHTC3 sensor\nmeasures both temperature\nand humidity.
+The Sensirion SHT21/SHTC3 sensors\nmeasure both temperature\nand humidity.
 Text Notes 7500 5000 0    157  ~ 0
 Button

Commit message: Upgrade file format
Parts:
- C1, C2, C3: symbol C -> backplane-rescue:C
- D1, D2, D3: symbol LED_Small -> backplane-rescue:LED_Small
- D4, D6: symbol D -> backplane-rescue:D
- D5: symbol D_Zener_Small -> backplane-rescue:D_Zener_Small
- F1: symbol Polyfuse_Small -> backplane-rescue:Polyfuse_Small
- J1, J2: symbol I2C_HEADER -> backplane-rescue:I2C_HEADER
- J3: symbol SERIAL_HEADER -> backplane-rescue:SERIAL_HEADER
- J4, J5: symbol PWR_HEADER -> backplane-rescue:PWR_HEADER
- J6: symbol FAN -> backplane-rescue:FAN
- J7: symbol Conn_01x01 -> backplane-rescue:Conn_01x01
- Q4: symbol Q_NMOS_GSD -> backplane-rescue:Q_NMOS_GSD
- Q5: symbol Q_PMOS_GSD -> backplane-rescue:Q_PMOS_GSD
- R1, R2, R3: symbol R-RESCUE-backplane -> backplane-rescue:R-RESCUE-backplane
- R10, R11, R12, R13, R4, R5, R9: symbol R -> backplane-rescue:R
- SW1: symbol SW_Push -> backplane-rescue:SW_Push
- U1: symbol Raspi_2_3 -> backplane-rescue:Raspi_2_3
- U2: symbol IC880A-SPI -> backplane-rescue:IC880A-SPI
- U3: symbol SHT21 -> backplane-rescue:SHT21
- U4: symbol MP1584_MODULE -> backplane-rescue:MP1584_MODULE
- U5: symbol MCP3425A0T-E/CH-RESCUE-backplane -> backplane-rescue:MCP3425A0T-E_CH-RESCUE-backplane
- U6: symbol SHTC3 -> backplane-rescue:SHTC3
